File: DAQ_design/v0.2.1/revB/revb/revb.kicad_sch (KiCad schematic)
At the start: 19 parts, among them Q1 BC549, Q2 IRF9540N, Q3 IRF540N, Q4 BC549, Q5 IRF9540N, Q6 IRF540N, U1 ADS1115IDGS

Commit message: revb changes
revb changes
Changed lines of the file:
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@@
   (symbol (lib_id "Device:R") (at 53.34 132.08 270) (unit 1)
     (in_bom yes) (on_board yes) (dnp no)
-    (property "Reference" "R8" (at 53.34 126.8222 90)
-      (effects (font (size 1.27 1.27)))
-    )
-    (property "Value" "1k" (at 53.34 129.1336 90)
+    (property "Reference" "R8" (at 48.26 128.27 90)
+      (effects (font (size 1.27 1.27)))
+    )
+    (property "Value" "1k" (at 46.99 137.16 90)
       (effects (font (size 1.27 1.27)))
     )
@@
       (effects (font (size 1.27 1.27)) hide)
     )
+    (pin "1")
+    (pin "10")
+    (pin "2")
+    (pin "3")
+    (pin "4")
     (pin "5")
-    (pin "3")
     (pin "6")
-    (pin "2")
     (pin "7")
     (pin "8")
     (pin "9")
-    (pin "10")
-    (pin "1")
-    (pin "4")
-    (instances
-      (project "revb"
+    (instances
+      (project "revb"

Commit message: updates to revb
graphics and traces
Connections:
- net VDD: now also Arduino1.27 (+5V)
Changed lines of the file:
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@@
+    )
+  )
+  (global_label "VDD" (shape input) (at 187.96 102.87 90)
+    (effects (font (size 1.27 1.27)) (justify left))
+    (property "Intersheetrefs" "${INTERSHEET_REFS}" (at 187.96 102.87 0)
+      (effects (font (size 1.27 1.27)) hide)
     )
   )
@@
     )
   )
+  (global_label "VDD" (shape input) (at 120.65 114.3 90)
+    (effects (font (size 1.27 1.27)) (justify left))
+    (property "Intersheetrefs" "${INTERSHEET_REFS}" (at 120.65 114.3 0)
+      (effects (font (size 1.27 1.27)) hide)
+    )
+  )
   (symbol (lib_id "Transistor_FET:IRF9540N") (at 110.49 69.85 0) (unit 1)
     (in_bom yes) (on_board yes) (dnp no)
@@
         )
       )
-    )
-  )
-  (symbol (lib_id "power:VDD") (at 187.96 102.87 0) (unit 1)
-    (in_bom yes) (on_board yes) (dnp no)
-    (property "Reference" "#PWR0114" (at 187.96 106.68 0)
-      (effects (font (size 1.27 1.27)) hide)
-    )
-    (property "Value" "VDD" (at 188.341 98.4758 0)
-      (effects (font (size 1.27 1.27)))
-    )
-    (property "Footprint" "" (at 187.96 102.87 0)
-      (effects (font (size 1.27 1.27)) hide)
-    )
-    (property "Datasheet" "" (at 187.96 102.87 0)
-      (effects (font (size 1.27 1.27)) hide)
-    )
-    (pin "1")
-    (instances
-      (project "revb"
-        (path "/1e50868d-c684-405d-aeb1-67a12047a543"
-          (reference "#PWR0114") (unit 1)
-        )
-      )

Commit message: start on revb fixes
Parts:
- R1, R2, R3, R4, R5, R6, R7, R8: footprint Resistor_SMD:R_0603_1608Metric -> Resistor_SMD:R_1206_3216Metric
Connections:
- net GND: now also U1.2 (GND); no longer Screw_Terminal1.1 (Pin_1), Screw_Terminal1.2 (Pin_2), Screw_Terminal1.3 (Pin_3), Screw_Terminal1.4 (Pin_4), U1.10 (AIN3), U1.7 (AIN0), U1.8 (AIN1), U1.9 (AIN2)
- new net AIN1: Screw_Terminal1.2 (Pin_2), U1.8 (AIN1)
- new net AIN2: Screw_Terminal1.3 (Pin_3), U1.9 (AIN2)
- new net AIN3: Screw_Terminal1.4 (Pin_4), U1.10 (AIN3)
- new net AN0: Screw_Terminal1.1 (Pin_1), U1.7 (AIN0)

Commit message: attempted fixes
Connections:
- net AIN1: now also Screw_Terminal1.3 (Pin_3); no longer Screw_Terminal1.2 (Pin_2)
- net AIN2: now also Screw_Terminal1.2 (Pin_2); no longer Screw_Terminal1.3 (Pin_3)
- net AIN3: now also Screw_Terminal1.1 (Pin_1); no longer Screw_Terminal1.4 (Pin_4)
- net AN0: now also Screw_Terminal1.4 (Pin_4); no longer Screw_Terminal1.1 (Pin_1)
Changed lines of the file:
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@@
     )
   )
-  (global_label "AN0" (shape input) (at 57.15 152.4 180)
+  (global_label "AN0" (shape input) (at 57.15 160.02 180)
     (effects (font (size 1.27 1.27)) (justify right))
-    (property "Intersheetrefs" "${INTERSHEET_REFS}" (at 57.15 152.4 0)
+    (property "Intersheetrefs" "${INTERSHEET_REFS}" (at 57.15 160.02 0)
       (effects (font (size 1.27 1.27)) hide)
     )
@@
     )
   )
-  (global_label "AIN3" (shape input) (at 57.15 160.02 180)
+  (global_label "AIN3" (shape input) (at 57.15 152.4 180)
     (effects (font (size 1.27 1.27)) (justify right))
-    (property "Intersheetrefs" "${INTERSHEET_REFS}" (at 57.15 160.02 0)
+    (property "Intersheetrefs" "${INTERSHEET_REFS}" (at 57.15 152.4 0)
       (effects (font (size 1.27 1.27)) hide)
     )
@@
     )
   )
-  (global_label "AIN2" (shape input) (at 57.15 157.48 180)
+  (global_label "AIN2" (shape input) (at 57.15 154.94 180)
     (effects (font (size 1.27 1.27)) (justify right))
-    (property "Intersheetrefs" "${INTERSHEET_REFS}" (at 57.15 157.48 0)
+    (property "Intersheetrefs" "${INTERSHEET_REFS}" (at 57.15 154.94 0)
       (effects (font (size 1.27 1.27)) hide)
     )
@@
     )
   )
-  (global_label "AIN1" (shape input) (at 57.15 154.94 180)
+  (global_label "AIN1" (shape input) (at 57.15 157.48 180)
     (effects (font (size 1.27 1.27)) (justify right))
-    (property "Intersheetrefs" "${INTERSHEET_REFS}" (at 57.15 154.94 0)
+    (property "Intersheetrefs" "${INTERSHEET_REFS}" (at 57.15 157.48 0)
       (effects (font (size 1.27 1.27)) hide)
     )
