File: DAQ_design/v0.2.1/CAD/faceplate_front/faceplate_front.kicad_pcb (KiCad board)
At the start: 2 copper layers, 78 x 42.9 mm, 5 parts

Commit message: more faceplate stuff
Parts:
- added G2: LOGO, uofsc_foots:uofsc, B.Cu at (138.7, 100.1)
- added G3: LOGO, uofsc_foots:upg, B.Cu at (149.7, 100.1)
- moved REF** 11.9 mm to (126.0, 103.3)
- moved REF** 11.9 mm to (126.0, 67.8)
- moved REF** 11.9 mm to (177.4, 85.7)
- moved REF** 11.9 mm to (196.1, 67.8)
- moved REF** 11.9 mm to (196.1, 103.3)
Routing:
- removed copper zone on F.Cu, net (none)
Other:
- outline, holes or cut-outs redrawn
- board text added: "5V"
- board text added: "Biphasic Data Acquisition System"
