File: DAQ_design/v0.2.1/CAD/faceplate_back/faceplate_back.kicad_pcb (KiCad board)
At the start: 2 copper layers, 78 x 42.9 mm, 7 parts

Commit message: more faceplate stuff
Parts:
- removed G2: LOGO, uofsc_foots:uofsc
- added REF**: DINRailAdapter_3xM3_PhoenixContact_1201578, MountingEquipment:DINRailAdapter_3xM3_PhoenixContact_1201578, F.Cu at (152.0, 78.0)
- added REF**: DINRailAdapter_3xM3_PhoenixContact_1201578, MountingEquipment:DINRailAdapter_3xM3_PhoenixContact_1201578, F.Cu at (145.5, 78.0)
Routing:
- removed copper zone on F.Cu, net (none)
Other:
- outline, holes or cut-outs redrawn
- board text added: "AIN0"
- board text added: "AIN1"
- board text added: "AIN2"
- board text added: "AIN3"
- board text added: "GND"
- board text added: "SN"
- board text added: "SP"

Commit message: begin redraw
Parts:
- moved REF** 0.42 mm to (172.0, 96.5)
Other:
- outline, holes or cut-outs redrawn
Changed lines of the file:
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@@
   )
   (footprint "MountingHole:MountingHole_3.2mm_M3" (layer "F.Cu")
-    (at 172.42 96.5)
+    (at 172 96.5)
     (descr "Mounting Hole 3.2mm, no annular, M3")
     (tags "mounting hole 3.2mm no annular m3")
@@
     )
   )
+  (gr_line (start 134 92) (end 134 90)
+    (stroke (width 0.05) (type default)) (layer "Edge.Cuts"))
   (gr_line (start 183.298 115.176) (end 113.32 115.176)
     (stroke (width 0.2) (type solid)) (layer "Edge.Cuts"))
   (gr_circle (center 183.361 111.493) (end 185.468265 111.493)
     (stroke (width 0.2) (type solid)) (fill none) (layer "Edge.Cuts"))
+  (gr_line (start 162 90) (end 162 92)
+    (stroke (width 0.05) (type default)) (layer "Edge.Cuts"))
   (gr_line (start 109.32 76.24) (end 109.32 111.186)
     (stroke (width 0.2) (type solid)) (layer "Edge.Cuts"))
-  (gr_rect (start 130 91.9) (end 168.4 101.2)
-    (stroke (width 0.05) (type default)) (fill none) (layer "Edge.Cuts"))
+  (gr_line (start 130 101.2) (end 130 92)
+    (stroke (width 0.05) (type default)) (layer "Edge.Cuts"))
+  (gr_line (start 168 101.2) (end 168 92)
+    (stroke (width 0.05) (type default)) (layer "Edge.Cuts"))
+  (gr_line (start 162 92) (end 136 92)
+    (stroke (width 0.05) (type default)) (layer "Edge.Cuts"))
   (gr_circle (center 183.361 75.933) (end 185.297331 75.933)
     (stroke (width 0.2) (type solid)) (fill none) (layer "Edge.Cuts"))
@@
   (gr_arc (start 187.298 111.186) (mid 186.129356 114.007356) (end 183.308 115.176)
     (stroke (width 0.2) (type solid)) (layer "Edge.Cuts"))
+  (gr_line (start 134 90) (end 136 90)
+    (stroke (width 0.05) (type default)) (layer "Edge.Cuts"))
   (gr_arc (start 109.32 76.24) (mid 110.488644 73.418644) (end 113.31 72.25)
     (stroke (width 0.2) (type solid)) (layer "Edge.Cuts"))
+  (gr_line (start 136 90) (end 136 92)
+    (stroke (width 0.05) (type default)) (layer "Edge.Cuts"))
+  (gr_line (start 130 92) (end 134 92)
+    (stroke (width 0.05) (type default)) (layer "Edge.Cuts"))
   (gr_line (start 187.298 111.186) (end 187.298 76.24)
     (stroke (width 0.2) (type solid)) (layer "Edge.Cuts"))
   (gr_line (start 183.308 72.25) (end 113.31 72.25)
     (stroke (width 0.2) (type solid)) (layer "Edge.Cuts"))
+  (gr_line (start 164 90) (end 162 90)
+    (stroke (width 0.05) (type default)) (layer "Edge.Cuts"))
+  (gr_line (start 130 101.2) (end 168 101.2)
+    (stroke (width 0.05) (type default)) (layer "Edge.Cuts"))
   (gr_circle (center 113.257 111.493) (end 115.236989 111.493)
     (stroke (width 0.2) (type solid)) (fill none) (layer "Edge.Cuts"))
@@
   (gr_line (start 187.298 76.25) (end 187.298 111.176)
     (stroke (width 0.2) (type solid)) (layer "Edge.Cuts"))
+  (gr_line (start 164 92) (end 164 90)
+    (stroke (width 0.05) (type default)) (layer "Edge.Cuts"))
+  (gr_line (start 168 92) (end 164 92)
+    (stroke (width 0.05) (type default)) (layer "Edge.Cuts"))
   (gr_circle (center 113.257 75.933) (end 115.323801 75.933)
     (stroke (width 0.2) (type solid)) (fill none) (layer "Edge.Cuts"))
@@
     (effects (font (size 0.75 0.75) (thickness 0.1875) bold) (justify left bottom))
   )
-  (zone (net 0) (net_name "") (layers "F.Cu" "F.Fab") (hatch edge 0.5)
-    (connect_pads (clearance 0))
-    (min_thickness 0.25) (filled_areas_thickness no)
-    (keepout (tracks not_allowed) (vias not_allowed) (pads not_allowed) (copperpour not_allowed) (footprints allowed))
-    (fill (thermal_gap 0.5) (thermal_bridge_width 0.5))
-    (polygon
-      (pts
-        (xy 129.93 91.86)
-        (xy 129.93 101.15)
-        (xy 168.4 101.14)
-        (xy 168.41 91.86)
-      )
-    )
-  )
 )
