File: DAQ_design/v0.2.1/CAD/biphasic_v0.2.1/biphasic_resized/biphasic_resized.kicad_pcb (KiCad board)
At the start: 2 copper layers, 119 x 75 mm, 25 parts, among them Q1 BC549, Q2 IRF9540N, Q3 IRF540N, Q4 BC549, Q5 IRF540N, Q6 IRF9540N

Commit message: begin redraw
Parts:
- added J1: Conn_01x03_Pin, Connector_PinHeader_2.54mm:PinHeader_1x03_P2.54mm_Vertical, F.Cu at (207.0, 110.9)
Other:
- board text added: "10Hz"
- board text added: "5Hz"
Changed lines of the file:
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@@
   (net 4 "Net-(ADC1-SCL)")
   (net 5 "Net-(ADC1-SDA)")
-  (net 6 "unconnected-(ADC1-ALERT{slash}RDY-Pad6)")
+  (net 6 "Net-(Arduino1-D2)")
   (net 7 "AIN0")
   (net 8 "AIN1")
@@
   (net 12 "unconnected-(Arduino1-RX1-Pad2)")
   (net 13 "Net-(Arduino1-~{RESET}-Pad3)")
-  (net 14 "unconnected-(Arduino1-D2-Pad5)")
-  (net 15 "unconnected-(Arduino1-D3-Pad6)")
+  (net 14 "Net-(Arduino1-D3)")
+  (net 15 "Net-(Arduino1-D4)")
   (net 16 "unconnected-(Arduino1-D4-Pad7)")
   (net 17 "unconnected-(Arduino1-D5-Pad8)")
@@
   (net 39 "Net-(Q4-C)")
   (net 40 "Net-(Q4-B)")
+  (net 41 "unconnected-(Arduino1-D3-Pad6)")
+  (net 42 "unconnected-(Arduino1-D2-Pad5)")
+  (net 43 "unconnected-(ADC1-ALERT{slash}RDY-Pad6)")
   (footprint "Resistor_SMD:R_1206_3216Metric" (layer "F.Cu")
     (at 151.5375 63.5375 90)
@@
       (net 2 "GND") (pinfunction "ADDR") (pintype "input"))
     (pad "6" thru_hole circle (at 15.24 -2.032 90) (size 2 2) (drill 1) (layers "*.Cu" "*.Mask")
-      (net 6 "unconnected-(ADC1-ALERT{slash}RDY-Pad6)") (pinfunction "ALERT/RDY") (pintype "output"))
+      (net 43 "unconnected-(ADC1-ALERT{slash}RDY-Pad6)") (pinfunction "ALERT/RDY") (pintype "output"))
     (pad "7" thru_hole circle (at 17.78 -2.032 90) (size 2 2) (drill 1) (layers "*.Cu" "*.Mask")
       (net 7 "AIN0") (pinfunction "AIN0") (pintype "input"))
@@
       (stroke (width 0) (type solid)) (fill solid) (layer "F.SilkS"))
   )
+  (footprint "Connector_PinHeader_2.54mm:PinHeader_1x03_P2.54mm_Vertical" (layer "F.Cu")
+    (at 207 110.92)
+    (descr "Through hole straight pin header, 1x03, 2.54mm pitch, single row")
+    (tags "Through hole pin header THT 1x03 2.54mm single row")
+    (property "Sheetfile" "biphasic_resized.kicad_sch")
+    (property "Sheetname" "")
+    (property "ki_description" "Generic connector, single row, 01x03, script generated")
+    (property "ki_keywords" "connector")
+    (attr through_hole)
+    (fp_text reference "J1" (at 0 -2.33) (layer "F.SilkS")
+        (effects (font (size 1 1) (thickness 0.15)))
+    )
+    (fp_text value "Conn_01x03_Pin" (at 0 7.41) (layer "F.Fab")
+        (effects (font (size 1 1) (thickness 0.15)))
+    )
+    (fp_text user "${REFERENCE}" (at 0 2.54 90) (layer "F.Fab")
+        (effects (font (size 1 1) (thickness 0.15)))
+    )
+    (fp_line (start -1.33 -1.33) (end 0 -1.33)
+      (stroke (width 0.12) (type solid)) (layer "F.SilkS"))
+    (fp_line (start -1.33 0) (end -1.33 -1.33)
+      (stroke (width 0.12) (type solid)) (layer "F.SilkS"))
+    (fp_line (start -1.33 1.27) (end -1.33 6.41)
+      (stroke (width 0.12) (type solid)) (layer "F.SilkS"))
+    (fp_line (start -1.33 1.27) (end 1.33 1.27)
+      (stroke (width 0.12) (type solid)) (layer "F.SilkS"))
+    (fp_line (start -1.33 6.41) (end 1.33 6.41)
+      (stroke (width 0.12) (type solid)) (layer "F.SilkS"))
+    (fp_line (start 1.33 1.27) (end 1.33 6.41)
+      (stroke (width 0.12) (type solid)) (layer "F.SilkS"))
+    (fp_line (start -1.8 -1.8) (end -1.8 6.85)
+      (stroke (width 0.05) (type solid)) (layer "F.CrtYd"))
+    (fp_line (start -1.8 6.85) (end 1.8 6.85)
+      (stroke (width 0.05) (type solid)) (layer "F.CrtYd"))
+    (fp_line (start 1.8 -1.8) (end -1.8 -1.8)
+      (stroke (width 0.05) (type solid)) (layer "F.CrtYd"))
+    (fp_line (start 1.8 6.85) (end 1.8 -1.8)
+      (stroke (width 0.05) (type solid)) (layer "F.CrtYd"))
+    (fp_line (start -1.27 -0.635) (end -0.635 -1.27)
+      (stroke (width 0.1) (type solid)) (layer "F.Fab"))
+    (fp_line (start -1.27 6.35) (end -1.27 -0.635)
+      (stroke (width 0.1) (type solid)) (layer "F.Fab"))
+    (fp_line (start -0.635 -1.27) (end 1.27 -1.27)
+      (stroke (width 0.1) (type solid)) (layer "F.Fab"))
+    (fp_line (start 1.27 -1.27) (end 1.27 6.35)
+      (stroke (width 0.1) (type solid)) (layer "F.Fab"))
+    (fp_line (start 1.27 6.35) (end -1.27 6.35)
+      (stroke (width 0.1) (type solid)) (layer "F.Fab"))
+    (pad "1" thru_hole rect (at 0 0) (size 1.7 1.7) (drill 1) (layers "*.Cu" "*.Mask")
+      (net 6 "Net-(Arduino1-D2)") (pinfunction "Pin_1") (pintype "passive"))
+    (pad "2" thru_hole oval (at 0 2.54) (size 1.7 1.7) (drill 1) (layers "*.Cu" "*.Mask")
+      (net 14 "Net-(Arduino1-D3)") (pinfunction "Pin_2") (pintype "passive"))
+    (pad "3" thru_hole oval (at 0 5.08) (size 1.7 1.7) (drill 1) (layers "*.Cu" "*.Mask")
+      (net 15 "Net-(Arduino1-D4)") (pinfunction "Pin_3") (pintype "passive"))
+    (model "/home/david/Documents/GitHub/Biphasic-data-acquisition-system/DAQ_design/v0.2.1/CAD/biphasic_v0.2.1/stp_files/pinheader 1x3 and 1 jumper.stp"
+      (offset (xyz 0 17.5 0))
+      (scale (xyz 1 1 1))
+      (rotate (xyz 0 0 90))
+    )
+  )
   (footprint "Connector_BarrelJack:BarrelJack_Horizontal" (layer "F.Cu")
     (at 135 70)
@@
       (net 2 "GND") (pinfunction "GND") (pintype "power_in"))
     (pad "5" thru_hole oval (at 0 10.16 270) (size 1.6 1.6) (drill 1) (layers "*.Cu" "*.Mask")
-      (net 14 "unconnected-(Arduino1-D2-Pad5)") (pinfunction "D2") (pintype "bidirectional"))
+      (net 42 "unconnected-(Arduino1-D2-Pad5)") (pinfunction "D2") (pintype "bidirectional"))
     (pad "6" thru_hole oval (at 0 12.7 270) (size 1.6 1.6) (drill 1) (layers "*.Cu" "*.Mask")
-      (net 15 "unconnected-(Arduino1-D3-Pad6)") (pinfunction "D3") (pintype "bidirectional"))
+      (net 41 "unconnected-(Arduino1-D3-Pad6)") (pinfunction "D3") (pintype "bidirectional"))
     (pad "7" thru_hole oval (at 0 15.24 270) (size 1.6 1.6) (drill 1) (layers "*.Cu" "*.Mask")
       (net 16 "unconnected-(Arduino1-D4-Pad7)") (pinfunction "D4") (pintype "bidirectional"))
@@
   (gr_line (start 240 49) (end 121 49)
     (stroke (width 0.1) (type default)) (layer "Edge.Cuts"))
+  (gr_text "5Hz" (at 209 113) (layer "F.SilkS")
+    (effects (font (size 1 1) (thickness 0.15)) (justify left bottom))
+  )
   (gr_text "H.B. Birgin\nDavid Wamai\nJoud Satme\nAustin R.J. Downey" (at 164 120) (layer "F.SilkS")
     (effects (font (size 1 1) (thickness 0.1)) (justify bottom))
   )
+  (gr_text "10Hz" (at 209 116) (layer "F.SilkS")
+    (effects (font (size 1 1) (thickness 0.15)) (justify left bottom))
+  )
   (segment (start 155.14 101.76) (end 149.14 101.76) (width 0.25) (layer "F.Cu") (net 3))

Commit message: sync
Parts:
- removed J1: Conn_01x03_Pin, Connector_PinHeader_2.54mm:PinHeader_1x03_P2.54mm_Vertical
Other:
- board text removed: "10Hz"
- board text removed: "5Hz"
