File: DAQ_design/v0.2.1/CAD/v0.2.1/v0.2.1.kicad_sch (KiCad schematic)
At the start: 2 parts, among them U1 Teensy4.0, U2 TLV6001DCK

Commit message: new code and cad
Parts:
- removed U2: TLV6001DCK, Package_TO_SOT_SMD:SOT-353_SC-70-5, symbol Amplifier_Operational:TLV6001DCK
- added C1: 1uF, symbol Device:C_Small
- added FB1, FB2: MMZ2012Y152B, symbol Device:FerriteBead_Small
- added R1: 10k, symbol Device:R_Small
- added R2: 10K, symbol Device:R_Small
- added U2: L293, Package_DIP:DIP-16_W7.62mm, symbol Driver_Motor:L293
- added U3: LM324, symbol Amplifier_Operational:LM324
- added U4: ADS1115IDGS, Package_SO:TSSOP-10_3x3mm_P0.5mm, symbol Analog_ADC:ADS1115IDGS
Connections:
- net GND: now reaches U1.1 (GND)
- net GND: now also FB2.2, U4.1 (ADDR)
- net IN1: now reaches U1.2 (0_RX1_CRX2_CS1)
- net IN1: now also U2.2 (1A), U4.5 (AIN1)
- net IN2: now reaches U1.3 (1_TX1_CTX2_MISO1)
- net IN2: now also U2.7 (2A), U4.6 (AIN2)
- net PWM: no longer names the net of U1.52 (39_DAT2_TX5)
- new net: C1.2, FB2.1, U4.3 (GND)
- new net: U2.3 (1Y), U3.3 (+)
- new net: C1.1, FB1.2, U4.8 (VDD)
- new net ADC_SCL: R1.2, R2.2, U4.10 (SCL), U4.9 (SDA)
- new net EX+: U3.1, U3.2 (-)
- new net EX-: U2.6 (2Y)
- new net IN0: U4.4 (AIN0)
- new net IN3: U4.7 (AIN3)
- new net VDD: FB1.1, R1.1, R2.1

Commit message: pushing test figures
Parts:
- removed U3: LM324, symbol Amplifier_Operational:LM324
- added A1: SD_Card_Module, Charleslabs_Parts:SD_Card_Module, symbol Charleslabs_Parts:SD_Card_Module
- added J1: Screw_Terminal_01x04, symbol Connector:Screw_Terminal_01x04
Connections:
- net ADC_SCL: now also U1.25 (18_A4_SDA0), U1.26 (19_A5_SCL0)
- net EX+: now also U2.3 (1Y), J1.3 (Pin_3)
- net EX-: now also J1.4 (Pin_4)
- net GND: now also U1.17 (GND), U2.12 (GND), U2.13 (GND), U2.4 (GND), U2.5 (GND), A1.6 (GND)
- net IN0: now also J1.1 (Pin_1)
- net IN1: now also J1.2 (Pin_2)
- net SDCS: now reaches U1.12 (10_CS_MQSR)
- net SDCS: now also A1.2 (CS)
- net SDMOSI: now reaches U1.13 (11_MOSI_CTX1)
- net SDMOSI: now also A1.3 (MOSI)
- net SDMISO: now reaches U1.14 (12_MISO_MQSL)
- net SDMISO: now also A1.5 (MISO)
- net SDCLK: now reaches U1.20 (13_SCK_CRX1_LED)
- net SDCLK: now also A1.4 (CLK)
- net +3.3V: now reaches U1.31 (3V3)
- net +3.3V: now also A1.1 (3V3)

Commit message: tests and cad
Parts:
- removed U2: L293, Package_DIP:DIP-16_W7.62mm, symbol Driver_Motor:L293
- added 5V1: Barrel_Jack, Connector_BarrelJack:BarrelJack_Horizontal, symbol Connector:Barrel_Jack
- added D1: zener1, Diode_SMD:D_1206_3216Metric, symbol Device:D_Zener_Small
- added D2: zener2, Diode_SMD:D_1206_3216Metric, symbol Device:D_Zener_Small
- added D3: zener3, Diode_SMD:D_1206_3216Metric, symbol Device:D_Zener_Small
- added D4: zener4, Diode_SMD:D_1206_3216Metric, symbol Device:D_Zener_Small
- added D5, D6: LED, LED_SMD:LED_1206_3216Metric, symbol Device:LED
- added Q1, Q4: BC549, Package_TO_SOT_THT:TO-92_Inline_Wide, symbol Transistor_BJT:BC549
- added Q2, Q6: IRF9540N, Package_TO_SOT_THT:TO-220-3_Vertical, symbol Transistor_FET:IRF9540N
- added Q3, Q5: IRF540N, Package_TO_SOT_THT:TO-220-3_Vertical, symbol Transistor_FET:IRF540N
- added R10, R11, R9: R_Small, Resistor_SMD:R_1206_3216Metric, symbol Device:R_Small
- added R3, R5: 1k, Resistor_SMD:R_1206_3216Metric, symbol Device:R
- added R4, R6: 10k, Resistor_SMD:R_1206_3216Metric, symbol Device:R
- added R7, R8: 260, Resistor_SMD:R_1206_3216Metric, symbol Device:R
- added U2, U3: SFH617A-1X001, Package_DIP:DIP-4_W7.62mm, symbol Isolator:SFH617A-1X001
- C1: footprint (none) -> Capacitor_SMD:C_1206_3216Metric
- FB1, FB2: footprint (none) -> Inductor_SMD:L_Ferrocore_DLG-0302
- J1: footprint (none) -> TerminalBlock:TerminalBlock_bornier-4_P5.08mm
- R1, R2: footprint (none) -> Resistor_SMD:R_1206_3216Metric
- U1: footprint (none) -> teensy.pretty-master:Teensy40
Connections:
- net ADC_SCL: no longer R2.2, U1.25 (18_A4_SDA0), U4.9 (SDA)
- net EX+: now also U4.6 (AIN2), D3.1 (K), R9.2; no longer J1.3 (Pin_3)
- net GND: now also U1.32 (GND), 5V1.2, D1.2 (A), D2.2 (A), D3.2 (A), D4.2 (A), Q1.3 (E), Q3.3 (S), Q4.3 (E), Q5.3 (S), R7.1, R8.1, U2.2, U2.3, U3.2, U3.3
- net IN0: now also D1.1 (K)
- net IN1: now also D2.1 (K); no longer U1.2 (0_RX1_CRX2_CS1)
- net IN3: now also J1.3 (Pin_3), D4.1 (K), R9.1
- net LEDPOW: now reaches U1.4 (2_OUT2)
- net LEDPOW: now also D5.2 (A)
- net LEDACT: now reaches U1.5 (3_LRCLK2)
- net LEDACT: now also D6.2 (A)
- net IN2 renamed LOGIC2
- net LOGIC2: now also R11.2; no longer U4.6 (AIN2)
- new net: Q4.1 (C), Q6.1 (G), R6.2
- new net: R10.1, U2.1
- new net: Q1.1 (C), Q2.1 (G), R4.2
- new net: Q1.2 (B), R3.1
- new net: D5.1 (K), R7.2
- new net: R11.1, U3.1
- new net: Q4.2 (B), R5.1
- new net: D6.1 (K), R8.2
- new net ADC_SDA: R2.2, U1.25 (18_A4_SDA0), U4.9 (SDA)
- new net LOGIC1: R10.2, U1.2 (0_RX1_CRX2_CS1)
- new net OPT1: Q5.1 (G), R3.2, U2.4
- new net OPT2: Q3.1 (G), R5.2, U3.4
- new net SN: Q5.2 (D), Q6.2 (D)
- new net SP: Q2.2 (D), Q3.2 (D)
- new net VPP: 5V1.1, Q2.3 (S), Q6.3 (S), R4.1, R6.1
Other:
- moved on the sheet: C1, FB1, FB2, J1, R1, R2, U4

Commit message: more cad
Parts:
- removed FB1, FB2: MMZ2012Y152B, Inductor_SMD:L_Ferrocore_DLG-0302, symbol Device:FerriteBead_Small
- removed Q1, Q4: BC549, Package_TO_SOT_THT:TO-92_Inline_Wide, symbol Transistor_BJT:BC549
- removed Q2, Q6: IRF9540N, Package_TO_SOT_THT:TO-220-3_Vertical, symbol Transistor_FET:IRF9540N
- removed Q3, Q5: IRF540N, Package_TO_SOT_THT:TO-220-3_Vertical, symbol Transistor_FET:IRF540N
- removed R3, R5: 1k, Resistor_SMD:R_1206_3216Metric, symbol Device:R
- removed R4, R6: 10k, Resistor_SMD:R_1206_3216Metric, symbol Device:R
- removed U2, U3: SFH617A-1X001, Package_DIP:DIP-4_W7.62mm, symbol Isolator:SFH617A-1X001
- added C2: 0.1uf, Capacitor_SMD:C_1206_3216Metric, symbol Device:C_Small
- added R12, R13, R6: 10k, Resistor_SMD:R_1206_3216Metric, symbol Device:R_Small
- added R3, R4, R5: 470, Resistor_SMD:R_1206_3216Metric, symbol Device:R_Small
- added S1: DS01C-254-L-09BE, dip-switch:SW_DS01C-254-L-09BE, symbol DS01C-254-L-09BE:DS01C-254-L-09BE
- added U2: L293D, Package_DIP:DIP-16_W7.62mm, symbol Driver_Motor:L293D
- added U3, U5, U6: PC817, Package_DIP:DIP-4_W7.62mm, symbol Isolator:PC817
- C1: value 1uF -> 1uf
- R10, R11: value R_Small -> 10k
Connections:
- net EX+: now also U2.3 (1Y)
- net EX-: now also J1.3 (Pin_3), U2.6 (2Y); no longer J1.4 (Pin_4)
- net GND: now also C2.1, U2.12 (GND), U2.13 (GND), U2.4 (GND), U2.5 (GND), U3.3, U5.3, U6.3; no longer A1.6 (GND), D1.2 (A), D2.2 (A), D3.2 (A), D4.2 (A), R7.1, R8.1, U1.1 (GND), U1.17 (GND), U1.32 (GND), U4.1 (ADDR)
- net IN3: now also J1.4 (Pin_4); no longer J1.3 (Pin_3)
- net LEDACT: now also U1.6 (4_BCLK2); no longer U1.5 (3_LRCLK2)
- net LEDPOW: now also U1.5 (3_LRCLK2); no longer U1.4 (2_OUT2)
- net LOGIC1: now also U3.1; no longer R10.2
- net LOGIC2: now also U5.1; no longer R11.2
- net OPT1: now also R6.2, U2.2 (1A), U3.4
- net OPT2: now also R10.2, U2.7 (2A), U5.4
- net VDD: now also C1.2, U1.33 (VIN), U4.8 (VDD), R13.1
- net VPP: now also R10.1, R11.1, C2.2, R6.1, U2.16 (VCC1), U2.8 (VCC2)
- net GNDD: now reaches U4.3 (GND)
- net GNDD: now also A1.6 (GND), C1.1, D1.2 (A), D2.2 (A), D3.2 (A), D4.2 (A), R7.1, R8.1, U1.1 (GND), U1.17 (GND), U1.32 (GND), R12.1, R3.2, R4.2, R5.2; no longer C1.2
- net at U4.2 (ALERT/RDY): now also R13.2
- new net: R12.2, U4.1 (ADDR)
- new net: R4.1, U5.2
- new net: R5.1, U6.2
- new net: R3.1, U3.2
- new net EN: U1.4 (2_OUT2), U6.1
- new net OPTEN: R11.2, U2.1 (EN1,2), U6.4
Other:
- moved on the sheet: 5V1, D1, D2, D3, D4, D5, D6, J1, R1, R2, R7, R8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

Commit message: power planes
Parts:
- D1, D2, D3, D4: footprint Diode_SMD:D_1206_3216Metric -> Diode_THT:D_DO-35_SOD27_P7.62mm_Horizontal
- D5: footprint LED_SMD:LED_1206_3216Metric -> LED_THT:LED_D5.0mm_Horizontal_O1.27mm_Z3.0mm_IRGrey
- D6: footprint LED_SMD:LED_1206_3216Metric -> LED_THT:LED_D5.0mm_Horizontal_O1.27mm_Z3.0mm
- R9: footprint Resistor_SMD:R_1206_3216Metric -> Resistor_THT:R_Axial_DIN0204_L3.6mm_D1.6mm_P7.62mm_Horizontal
Connections:
- net EX+: now also D1.1 (K), U4.4 (AIN0); no longer D3.1 (K), U4.6 (AIN2)
- net IN1: now also J1.4 (Pin_4), R9.1; no longer J1.2 (Pin_2)
- net IN3: now also J1.2 (Pin_2); no longer J1.4 (Pin_4), R9.1
- removed net IN0: D1.1 (K), J1.1 (Pin_1), U4.4 (AIN0)
- new net IN2: D3.1 (K), J1.1 (Pin_1), U4.6 (AIN2)
Changed lines of the file:
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@@
 	(global_label "IN0"
 		(shape input)
-		(at 144.78 170.18 180)
+		(at 114.3 189.23 270)
 		(fields_autoplaced yes)
 		(effects
@@
 		)
 		(property "Intersheetrefs" "${INTERSHEET_REFS}"
-			(at 138.65 170.18 0)
+			(at 114.3 195.36 90)
 			(effects
 				(font
@@
 	(global_label "IN2"
 		(shape input)
-		(at 114.3 189.23 270)
+		(at 144.78 170.18 180)
 		(fields_autoplaced yes)
 		(effects
@@
 		)
 		(property "Intersheetrefs" "${INTERSHEET_REFS}"
-			(at 114.3 195.36 90)
+			(at 138.65 170.18 0)
 			(effects
 				(font
@@
 	(global_label "IN3"
 		(shape input)
-		(at 130.81 189.23 270)
+		(at 144.78 172.72 180)
 		(fields_autoplaced yes)
 		(effects
@@
 		)
 		(property "Intersheetrefs" "${INTERSHEET_REFS}"
-			(at 130.81 195.36 90)
+			(at 138.65 172.72 0)
 			(effects
 				(font
@@
 	(global_label "IN1"
 		(shape input)
-		(at 144.78 172.72 180)
+		(at 130.81 189.23 270)
 		(fields_autoplaced yes)
 		(effects
@@
 		)
 		(property "Intersheetrefs" "${INTERSHEET_REFS}"
-			(at 138.65 172.72 0)
+			(at 130.81 195.36 90)
 			(effects
 				(font
@@
 		(on_board yes)
 		(dnp no)
-		(fields_autoplaced yes)
 		(property "Reference" "A1"
 			(at 139.7 39.3699 0)
@@
 		)
 		(property "Value" "SD_Card_Module"
-			(at 139.7 41.9099 0)
+			(at 139.446 42.672 0)
 			(effects
 				(font
@@
 			)
 		)
-		(property "Footprint" "Diode_SMD:D_1206_3216Metric"
+		(property "Footprint" "Diode_THT:D_DO-35_SOD27_P7.62mm_Horizontal"
 			(at 33.02 175.26 90)
 			(effects
@@
 			)
 		)
-		(property "Footprint" "Resistor_SMD:R_1206_3216Metric"
+		(property "Footprint" "Resistor_THT:R_Axial_DIN0204_L3.6mm_D1.6mm_P7.62mm_Horizontal"
 			(at 121.92 177.8 0)
 			(effects
@@
 			)
 		)
-		(property "Footprint" "Diode_SMD:D_1206_3216Metric"
+		(property "Footprint" "Diode_THT:D_DO-35_SOD27_P7.62mm_Horizontal"
 			(at 27.94 168.91 90)
 			(effects
@@
 			)
 		)
-		(property "Footprint" "LED_SMD:LED_1206_3216Metric"
+		(property "Footprint" "LED_THT:LED_D5.0mm_Horizontal_O1.27mm_Z3.0mm"
 			(at 269.24 134.62 0)
 			(effects
@@
 			)
 		)
-		(property "Footprint" "Diode_SMD:D_1206_3216Metric"
+		(property "Footprint" "Diode_THT:D_DO-35_SOD27_P7.62mm_Horizontal"
 			(at 38.1 181.61 90)
 			(effects
@@
 			)
 		)
-		(property "Footprint" "Diode_SMD:D_1206_3216Metric"
+		(property "Footprint" "Diode_THT:D_DO-35_SOD27_P7.62mm_Horizontal"
 			(at 43.18 187.96 90)
 			(effects
@@
 			)
 		)
-		(property "Footprint" "LED_SMD:LED_1206_3216Metric"
+		(property "Footprint" "LED_THT:LED_D5.0mm_Horizontal_O1.27mm_Z3.0mm_IRGrey"
 			(at 269.24 125.73 0)
 			(effects

Commit message: sync
Parts:
- added C3: 0.1uf, Capacitor_SMD:C_1206_3216Metric, symbol Device:C_Small
- added U7: 74HC165, Package_DIP:DIP-16_W7.62mm, symbol 74xx:74HC165
Connections:
- net +3.3V: now also U1.49 (3V3), C3.2, U7.16 (VCC)
- net GNDD: now also C3.1, U7.8 (GND)
- net LOGIC1: now also U1.10 (8_TX2_IN1); no longer U1.2 (0_RX1_CRX2_CS1)
- net LOGIC2: now also U1.11 (9_OUT1C); no longer U1.3 (1_TX1_CTX2_MISO1)
- net DIPDAT: now reaches U1.7 (5_IN2)
- net DIPDAT: now also U7.10 (DS)
- net DIPLAT: now reaches U1.8 (6_OUT1D)
- net DIPLAT: now also U7.1 (~{PL})
- net DIPCP: now reaches U1.9 (7_RX2_OUT1A)
- net DIPCP: now also U7.2 (CP)
- net SW1: now reaches S1.1B
- net SW1: now also U7.11 (D0)
- net SW2: now reaches S1.2B
- net SW2: now also U7.12 (D1)
- net SW3: now reaches S1.3B
- net SW3: now also U7.13 (D2)
- net SW4: now reaches S1.4B
- net SW4: now also U7.14 (D3)
- net SW5: now reaches S1.5B
- net SW5: now also U7.3 (D4)
- net SW6: now reaches S1.6B
- net SW6: now also U7.4 (D5)
- net SW7: now reaches S1.7B
- net SW7: now also U7.5 (D6)
- net SW8: now reaches S1.8B
- net SW8: now also U7.6 (D7)
Other:
- moved on the sheet: S1

Commit message: cad change sync
Connections:
- net SW1: now also S1.1A; no longer S1.1B
- net SW2: now also S1.2A; no longer S1.2B
- net SW3: now also S1.3A; no longer S1.3B
- net SW4: now also S1.4A; no longer S1.4B
- net SW5: now also S1.5A; no longer S1.5B
- net SW6: now also S1.6A; no longer S1.6B
- net SW7: now also S1.7A; no longer S1.7B
- net SW8: now also S1.8A; no longer S1.8B
Changed lines of the file:
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@@
 		(lib_id "DS01C-254-L-09BE:DS01C-254-L-09BE")
 		(at 217.17 124.46 0)
-		(mirror y)
 		(unit 1)
 		(exclude_from_sim no)

Commit message: 74hc165
Parts:
- removed S1: DS01C-254-L-09BE, dip-switch:SW_DS01C-254-L-09BE, symbol DS01C-254-L-09BE:DS01C-254-L-09BE
- added R14, R15, R16, R17, R18, R19, R20, R21, R22: 10k, Resistor_SMD:R_1206_3216Metric, symbol Device:R_Small
- added S1: DS03-254-10BE, dip-switch:SW_DS03-254-10BE, symbol DS03-254-10BE:DS03-254-10BE
- D5: footprint LED_THT:LED_D5.0mm_Horizontal_O1.27mm_Z3.0mm_IRGrey -> LED_SMD:LED_1206_3216Metric_Pad1.42x1.75mm_HandSolder
- D6: footprint LED_THT:LED_D5.0mm_Horizontal_O1.27mm_Z3.0mm -> LED_SMD:LED_1206_3216Metric_Pad1.42x1.75mm_HandSolder
Connections:
- net SW1 is gone; now on net VDD: U7.11 (D0)
- net SW2 is gone; now on net VDD: U7.12 (D1)
- net SW3 is gone; now on net VDD: U7.13 (D2)
- net SW4 is gone; now on net VDD: U7.14 (D3)
- net SW5 is gone; now on net VDD: U7.3 (D4)
- net SW6 is gone; now on net VDD: U7.4 (D5)
- net SW7 is gone; now on net VDD: U7.5 (D6)
- net SW8 is gone; now on net VDD: U7.6 (D7)
- net +3.3V: now also U1.16 (3V3); no longer C3.2, U7.16 (VCC)
- net DIPDAT: now also U7.9 (Q7); no longer U7.10 (DS)
- net GNDD: now also U7.10 (DS), U7.15 (~{CE}), R14.1, R15.1, R16.1, R17.1, R18.1, R19.1, R20.1, R21.1, R22.1
- net VDD: now also C3.2, U7.16 (VCC), S1.1A, S1.2A, S1.3A, S1.4A, S1.5A, S1.6A, S1.7A, S1.8A
- new net: R16.2, S1.3B
- new net: R18.2, S1.5B
- new net: R21.2, S1.8B
- new net: R17.2, S1.4B
- new net: R20.2, S1.7B
- new net: R22.2, S1.9B
- new net: R14.2, S1.1B
- new net: R15.2, S1.2B
- new net: R19.2, S1.6B
Other:
- moved on the sheet: C3, U7
