File: DAQ_design/v0.2.1/CAD/v0.2.1/v0.2.1.kicad_sch (KiCad schematic)
At the start: 42 parts, among them J1 Screw_Terminal_01x04, U1 Teensy4.0, U2 L293D, U3 PC817, U4 ADS1115IDGS, U5 PC817, U6 PC817, U7 74HC165

Commit message: routing progress
Parts:
- removed R22: 10k, Resistor_SMD:R_1206_3216Metric, symbol Device:R_Small
- R14, R15, R16, R17, R18, R19, R20, R21: footprint Resistor_SMD:R_1206_3216Metric -> Resistor_SMD:R_0805_2012Metric
Connections:
- net VDD: no longer U7.11 (D0), U7.12 (D1), U7.13 (D2), U7.14 (D3), U7.3 (D4), U7.4 (D5), U7.5 (D6), U7.6 (D7)
- net SW6: now reaches R16.2, S1.3B
- net SW6: now also U7.4 (D5)
- net SW4: now reaches R18.2, S1.5B
- net SW4: now also U7.14 (D3)
- net SW1: now reaches R21.2, S1.8B
- net SW1: now also U7.11 (D0)
- net SW5: now reaches R17.2, S1.4B
- net SW5: now also U7.3 (D4)
- net SW2: now reaches R20.2, S1.7B
- net SW2: now also U7.12 (D1)
- net SW8: now reaches R14.2, S1.1B
- net SW8: now also U7.6 (D7)
- net SW7: now reaches R15.2, S1.2B
- net SW7: now also U7.5 (D6)
- net SW3: now reaches R19.2, S1.6B
- net SW3: now also U7.13 (D2)
Other:
- moved on the sheet: R14, R15, R16, R17, R18, R19, R20, R21

Commit message: update v0.2.1 cad
Parts:
- removed C1: 1uf, Capacitor_SMD:C_1206_3216Metric, symbol Device:C_Small
- removed D1: zener1, Diode_THT:D_DO-35_SOD27_P7.62mm_Horizontal, symbol Device:D_Zener_Small
- removed D2: zener2, Diode_THT:D_DO-35_SOD27_P7.62mm_Horizontal, symbol Device:D_Zener_Small
- removed D3: zener3, Diode_THT:D_DO-35_SOD27_P7.62mm_Horizontal, symbol Device:D_Zener_Small
- removed D4: zener4, Diode_THT:D_DO-35_SOD27_P7.62mm_Horizontal, symbol Device:D_Zener_Small
- removed R1, R12, R13: 10k, Resistor_SMD:R_1206_3216Metric, symbol Device:R_Small
- removed R2: 10K, Resistor_SMD:R_1206_3216Metric, symbol Device:R_Small
- removed S1: DS03-254-10BE, dip-switch:SW_DS03-254-10BE, symbol DS03-254-10BE:DS03-254-10BE
- removed U4: ADS1115IDGS, Package_SO:TSSOP-10_3x3mm_P0.5mm, symbol Analog_ADC:ADS1115IDGS
- added A2: ADS1115_ADC_Module, Charleslabs_Parts:ADC1115_ADC_Module, symbol Charleslabs_Parts:ADS1115_ADC_Module
- added D10: zener4, Diode_THT:D_DO-35_SOD27_P7.62mm_Horizontal, symbol Device:D_Zener_Small
- added D7: zener1, Diode_THT:D_DO-35_SOD27_P7.62mm_Horizontal, symbol Device:D_Zener_Small
- added D8: zener2, Diode_THT:D_DO-35_SOD27_P7.62mm_Horizontal, symbol Device:D_Zener_Small
- added D9: zener3, Diode_THT:D_DO-35_SOD27_P7.62mm_Horizontal, symbol Device:D_Zener_Small
- added R22: 10k, Resistor_SMD:R_1206_3216Metric, symbol Device:R_Small
- added S2: 76PSB08ST, 8-pos-dip-switch-foot:76PSB08ST, symbol 8-pos-dip-switch:76PSB08ST
Connections:
- net ADC_SCL: now also A2.3 (SCL)
- net ADC_SDA: now also A2.4 (SDA)
- net EX+: now also A2.7 (A0), D7.1 (K)
- net GNDD: now also A2.2 (GND), D10.2 (A), D7.2 (A), D8.2 (A), D9.2 (A), R22.2
- net IN1: now also A2.8 (A1), D8.1 (K)
- net IN2: now also A2.9 (A2), D9.1 (K)
- net IN3: now also A2.10 (A3), D10.1 (K)
- net SW1: now also S2.B8 (COM_8)
- net SW2: now also S2.B7 (COM_7)
- net SW3: now also S2.B6 (COM_6)
- net SW4: now also S2.B5 (COM_5)
- net SW5: now also S2.B4 (COM_4)
- net SW6: now also S2.B3 (COM_3)
- net SW7: now also S2.B2 (COM_2)
- net SW8: now also S2.B1 (COM_1)
- net VDD: now also A2.1 (VCC), S2.A1 (NC_1), S2.A2 (NC_2), S2.A3 (NC_3), S2.A4 (NC_4), S2.A5 (NC_5), S2.A6 (NC_6), S2.A7 (NC_7), S2.A8 (NC_8)
- new net: A2.5 (ADDR), R22.1
Other:
- moved on the sheet: C3, R14, R15, R16, R17, R18, R19, R20, R21, U7

Commit message: i am a moron
Parts:
- D10, D7, D8, D9: footprint Diode_THT:D_DO-35_SOD27_P7.62mm_Horizontal -> Diode_SMD:D_1206_3216Metric_Pad1.42x1.75mm_HandSolder
- R22: footprint Resistor_SMD:R_1206_3216Metric -> Resistor_SMD:R_0805_2012Metric
Changed lines of the file:
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@@
 			)
 		)
-		(property "Footprint" "Diode_THT:D_DO-35_SOD27_P7.62mm_Horizontal"
+		(property "Footprint" "Diode_SMD:D_1206_3216Metric_Pad1.42x1.75mm_HandSolder"
 			(at 50.8 172.72 90)
 			(effects
@@
 			)
 		)
-		(property "Footprint" "Diode_THT:D_DO-35_SOD27_P7.62mm_Horizontal"
+		(property "Footprint" "Diode_SMD:D_1206_3216Metric_Pad1.42x1.75mm_HandSolder"
 			(at 40.64 160.02 90)
 			(effects
@@
 			)
 		)
-		(property "Footprint" "Diode_THT:D_DO-35_SOD27_P7.62mm_Horizontal"
+		(property "Footprint" "Diode_SMD:D_1206_3216Metric_Pad1.42x1.75mm_HandSolder"
 			(at 45.72 166.37 90)
 			(effects
@@
 			)
 		)
-		(property "Footprint" "Resistor_SMD:R_1206_3216Metric"
+		(property "Footprint" "Resistor_SMD:R_0805_2012Metric"
 			(at 48.26 139.7 0)
 			(effects
@@
 			)
 		)
-		(property "Footprint" "Diode_THT:D_DO-35_SOD27_P7.62mm_Horizontal"
+		(property "Footprint" "Diode_SMD:D_1206_3216Metric_Pad1.42x1.75mm_HandSolder"
 			(at 55.88 179.07 90)
 			(effects

Commit message: figuring out battery
Parts:
- removed 5V1: Barrel_Jack, Connector_BarrelJack:BarrelJack_Horizontal, symbol Connector:Barrel_Jack
- added BT1: Battery, symbol Device:Battery
Connections:
- net GND: now also BT1.2 (-)
- net VPP: now also BT1.1 (+)
Changed lines of the file:
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@@
 	(wire
 		(pts
-			(xy 270.51 158.75) (xy 274.32 158.75)
-		)
-		(stroke
-			(width 0)
-			(type default)
-		)
-	)
-	(wire
-		(pts
 			(xy 139.7 100.33) (xy 139.7 102.87)
 		)
@@
 	(wire
 		(pts
-			(xy 270.51 153.67) (xy 274.32 153.67)
-		)
-		(stroke
-			(width 0)
-			(type default)
-		)
-	)
-	(wire
-		(pts
 			(xy 170.18 107.95) (xy 175.26 107.95)
 		)
@@
 	)
 	(symbol
-		(lib_id "power:VPP")
-		(at 274.32 153.67 0)
-		(unit 1)
-		(exclude_from_sim no)
-		(in_bom yes)
-		(on_board yes)
-		(dnp no)
-		(property "Reference" "#PWR017"
-			(at 274.32 157.48 0)
-			(effects
-				(font
-					(size 1.27 1.27)
-				)
-				(hide yes)
-			)
-		)
-		(property "Value" "VPP"
-			(at 274.701 149.2758 0)
-			(effects
-				(font
-					(size 1.27 1.27)
-				)
-			)
-		)
-		(property "Footprint" ""
-			(at 274.32 153.67 0)
-			(effects
-				(font
-					(size 1.27 1.27)
-				)
-				(hide yes)
-			)
-		)
-		(property "Datasheet" ""
-			(at 274.32 153.67 0)
-			(effects
-				(font
-					(size 1.27 1.27)
-				)
-				(hide yes)
-			)
-		)
-		(property "Description" ""
-			(at 274.32 153.67 0)
-			(effects
-				(font
-					(size 1.27 1.27)
-				)
-				(hide yes)
-			)
-		)
-		(pin "1"
-		)
-		(instances
-			(project "v0.2.1"
-				(path "/f5ecb7fa-5db2-4074-ab55-2fe6f1a25df0"
-					(reference "#PWR017")
-					(unit 1)
-				)
-			)
-		)
-	)
-	(symbol
 		(lib_id "74xx:74HC165")
 		(at 220.98 107.95 0)
@@
 	)
 	(symbol
+		(lib_id "power:GND")
+		(at 196.85 156.21 0)
+		(mirror y)
+		(unit 1)
+		(exclude_from_sim no)
+		(in_bom yes)
+		(on_board yes)
+		(dnp no)
+		(property "Reference" "#PWR02"
+			(at 196.85 162.56 0)
+			(effects
+				(font
+					(size 1.27 1.27)
+				)
+				(hide yes)
+			)
+		)
+		(property "Value" "GND"
+			(at 196.8501 160.02 90)
+			(effects
+				(font
+					(size 1.27 1.27)
+				)
+				(justify right)
+			)
+		)
+		(property "Footprint" ""
+			(at 196.85 156.21 0)
+			(effects
+				(font
+					(size 1.27 1.27)
+				)
+				(hide yes)
+			)
+		)
+		(property "Datasheet" ""
+			(at 196.85 156.21 0)
+			(effects
+				(font
+					(size 1.27 1.27)
+				)
+				(hide yes)
+			)
+		)
+		(property "Description" "Power symbol creates a global label with name \"GND\" , ground"
+			(at 196.85 156.21 0)
+			(effects
+				(font
+					(size 1.27 1.27)
+				)
+				(hide yes)
+			)
+		)
+		(pin "1"
+		)
+		(instances
+			(project "v0.2.1"
+				(path "/f5ecb7fa-5db2-4074-ab55-2fe6f1a25df0"
+					(reference "#PWR02")
+					(unit 1)
+				)
+			)
+		)
+	)
+	(symbol
 		(lib_id "power:GNDD")
 		(at 208.28 125.73 270)
@@
 	)
 	(symbol
-		(lib_id "Connector:Barrel_Jack")
-		(at 262.89 156.21 0)
-		(unit 1)
-		(exclude_from_sim no)
-		(in_bom yes)
-		(on_board yes)
-		(dnp no)
-		(property "Reference" "5V1"
-			(at 264.3378 147.955 0)
-			(effects
-				(font
-					(size 1.27 1.27)
-				)
-			)
-		)
-		(property "Value" "Barrel_Jack"
-			(at 264.3378 150.2664 0)
-			(effects
-				(font
-					(size 1.27 1.27)
-				)
-			)
-		)
-		(property "Footprint" "Connector_BarrelJack:BarrelJack_Horizontal"
-			(at 264.16 157.226 0)
-			(effects
-				(font
-					(size 1.27 1.27)
-				)
-				(hide yes)
-			)
-		)
-		(property "Datasheet" "~"
-			(at 264.16 157.226 0)
-			(effects
-				(font
-					(size 1.27 1.27)
-				)
-				(hide yes)
-			)
-		)
-		(property "Description" ""
-			(at 262.89 156.21 0)
-			(effects
-				(font
-					(size 1.27 1.27)
-				)
-				(hide yes)
-			)
-		)
-		(pin "1"
-		)
-		(pin "2"
-		)
-		(instances
-			(project "v0.2.1"
-				(path "/f5ecb7fa-5db2-4074-ab55-2fe6f1a25df0"
-					(reference "5V1")
-					(unit 1)
-				)
-			)
-		)
-	)
-	(symbol
 		(lib_id "power:GND")
 		(at 199.39 30.48 90)
@@
 	)
 	(symbol
+		(lib_id "power:VDD")
+		(at 196.85 146.05 0)
+		(unit 1)
+		(exclude_from_sim no)
+		(in_bom yes)
+		(on_board yes)
+		(dnp no)
+		(fields_autoplaced yes)
+		(property "Reference" "#PWR01"
+			(at 196.85 149.86 0)
+			(effects
+				(font
+					(size 1.27 1.27)
+				)
+				(hide yes)
+			)
+		)
+		(property "Value" "VPP"
+			(at 196.85 140.97 0)
+			(effects
+				(font
+					(size 1.27 1.27)
+				)
+			)
+		)
+		(property "Footprint" ""
+			(at 196.85 146.05 0)
+			(effects
+				(font
+					(size 1.27 1.27)
+				)
+				(hide yes)
+			)
+		)
+		(property "Datasheet" ""
+			(at 196.85 146.05 0)
+			(effects
+				(font
+					(size 1.27 1.27)
+				)
+				(hide yes)
+			)
+		)
+		(property "Description" "Power symbol creates a global label with name \"VDD\""
+			(at 196.85 146.05 0)
+			(effects
+				(font
+					(size 1.27 1.27)
+				)
+				(hide yes)
+			)
+		)
+		(pin "1"
+		)
+		(instances
+			(project "v0.2.1"
+				(path "/f5ecb7fa-5db2-4074-ab55-2fe6f1a25df0"
+					(reference "#PWR01")
+					(unit 1)
+				)
+			)
+		)
+	)
+	(symbol
 		(lib_id "power:GNDD")
 		(at 50.8 175.26 0)
@@
 	)
 	(symbol
-		(lib_id "power:GND")
-		(at 274.32 158.75 0)
-		(unit 1)
-		(exclude_from_sim no)
-		(in_bom yes)
-		(on_board yes)
-		(dnp no)
-		(property "Reference" "#PWR018"
-			(at 274.32 165.1 0)
-			(effects
-				(font
-					(size 1.27 1.27)
-				)
-				(hide yes)
-			)
-		)
-		(property "Value" "GND"
-			(at 274.447 163.1442 0)
-			(effects
-				(font
-					(size 1.27 1.27)
-				)
-			)
-		)
-		(property "Footprint" ""
-			(at 274.32 158.75 0)
-			(effects
-				(font
-					(size 1.27 1.27)
-				)
-				(hide yes)
-			)
-		)
-		(property "Datasheet" ""
-			(at 274.32 158.75 0)
-			(effects
-				(font
-					(size 1.27 1.27)
-				)
-				(hide yes)
-			)
-		)
-		(property "Description" ""
-			(at 274.32 158.75 0)
-			(effects
-				(font
-					(size 1.27 1.27)
-				)
-				(hide yes)
-			)
-		)
-		(pin "1"
-		)
-		(instances
-			(project "v0.2.1"
-				(path "/f5ecb7fa-5db2-4074-ab55-2fe6f1a25df0"
-					(reference "#PWR018")
-					(unit 1)
-				)
-			)
-		)
-	)
-	(symbol
 		(lib_id "Device:R_Small")
 		(at 177.8 100.33 270)
@@
 					(unit 1)
 				)
+			)
+		)
+	)
+	(symbol
+		(lib_id "Device:Battery")
+		(at 196.85 151.13 0)
+		(unit 1)
+		(exclude_from_sim no)
+		(in_bom yes)
+		(on_board yes)
+		(dnp no)
+		(fields_autoplaced yes)
+		(property "Reference" "BT1"
+			(at 200.66 149.2884 0)
+			(effects
+				(font
+					(size 1.27 1.27)
+				)
+				(justify left)
+			)
+		)
+		(property "Value" "Battery"
+			(at 200.66 151.8284 0)
+			(effects
+				(font
+					(size 1.27 1.27)
+				)
+				(justify left)
+			)
+		)
+		(property "Footprint" ""
+			(at 196.85 149.606 90)
+			(effects
+				(font
+					(size 1.27 1.27)
+				)
+				(hide yes)
+			)
+		)
+		(property "Datasheet" "~"
+			(at 196.85 149.606 90)
+			(effects
+				(font
+					(size 1.27 1.27)
+				)
+				(hide yes)
+			)
+		)
+		(property "Description" "Multiple-cell battery"
+			(at 196.85 151.13 0)
+			(effects
+				(font
+					(size 1.27 1.27)
+				)
+				(hide yes)
+			)
+		)
+		(pin "2"
+		)
+		(pin "1"
+		)
+		(instances
+			(project ""
+				(path "/f5ecb7fa-5db2-4074-ab55-2fe6f1a25df0"
+					(reference "BT1")
+					(unit 1)
+				)

Commit message: resync
Connections:
- net +3.3V: no longer U1.16 (3V3)
- net ADC_SCL: now also U1.23 (16_A2_RX4_SCL1); no longer U1.26 (19_A5_SCL0)
- net ADC_SDA: now also U1.24 (17_A3_TX4_SDA1); no longer U1.25 (18_A4_SDA0)
- net EX+: now also A2.10 (A3), D10.1 (K); no longer A2.7 (A0), D7.1 (K)
- net EX-: now also J1.2 (Pin_2); no longer J1.3 (Pin_3)
- net IN1: now also A2.9 (A2), D9.1 (K), J1.1 (Pin_1); no longer A2.8 (A1), D8.1 (K), J1.4 (Pin_4)
- net IN2: now also A2.7 (A0), D7.1 (K), J1.4 (Pin_4); no longer A2.9 (A2), D9.1 (K), J1.1 (Pin_1)
- net IN3: now also A2.8 (A1), D8.1 (K), J1.3 (Pin_3); no longer A2.10 (A3), D10.1 (K), J1.2 (Pin_2)
- net LOGIC1: now also U5.1; no longer U3.1
- net LOGIC2: now also U3.1; no longer U5.1
- net OPT1: now also U5.4; no longer U3.4
- net OPT2: now also U3.4; no longer U5.4
- net at U5.2: now also R3.1; no longer R4.1
- net at U3.2: now also R4.1; no longer R3.1
Other:
- moved on the sheet: R9, U3, U5
Changed lines of the file:
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@@
 	)
 	(junction
-		(at 139.7 105.41)
+		(at 130.81 170.18)
 		(diameter 0)
 		(color 0 0 0 0)
 	)
 	(junction
-		(at 180.34 102.87)
+		(at 139.7 105.41)
 		(diameter 0)
 		(color 0 0 0 0)
 	)
 	(junction
-		(at 55.88 152.4)
+		(at 180.34 102.87)
 		(diameter 0)
 		(color 0 0 0 0)
 	)
 	(junction
-		(at 261.62 73.66)
+		(at 55.88 152.4)
 		(diameter 0)
 		(color 0 0 0 0)
 	)
 	(junction
-		(at 114.3 177.8)
+		(at 261.62 73.66)
 		(diameter 0)
 		(color 0 0 0 0)
 	)
 	(junction
-		(at 130.81 177.8)
+		(at 114.3 170.18)
 		(diameter 0)
 		(color 0 0 0 0)
@@
 	(wire
 		(pts
-			(xy 124.46 177.8) (xy 130.81 177.8)
+			(xy 124.46 170.18) (xy 130.81 170.18)
 		)
 		(stroke
@@
 	(wire
 		(pts
-			(xy 130.81 177.8) (xy 130.81 189.23)
+			(xy 130.81 170.18) (xy 130.81 181.61)
 		)
 		(stroke
@@
 	(wire
 		(pts
-			(xy 107.95 177.8) (xy 114.3 177.8)
+			(xy 107.95 170.18) (xy 114.3 170.18)
 		)
 		(stroke
@@
 	(wire
 		(pts
+			(xy 130.81 170.18) (xy 144.78 170.18)
+		)
+		(stroke
+			(width 0)
+			(type default)
+		)
+	)
+	(wire
+		(pts
 			(xy 45.72 147.32) (xy 45.72 163.83)
 		)
@@
 	(wire
 		(pts
-			(xy 114.3 177.8) (xy 114.3 189.23)
+			(xy 114.3 170.18) (xy 114.3 181.61)
 		)
 		(stroke
@@
 	(wire
 		(pts
-			(xy 114.3 177.8) (xy 119.38 177.8)
+			(xy 114.3 170.18) (xy 119.38 170.18)
 		)
 		(stroke
@@
 		)
 	)
-	(wire
-		(pts
-			(xy 130.81 177.8) (xy 144.78 177.8)
-		)
-		(stroke
-			(width 0)
-			(type default)
-		)
-	)
 	(global_label "OPT1"
 		(shape input)
@@
 	(global_label "IN0"
 		(shape input)
-		(at 33.02 144.78 180)
+		(at 33.02 152.4 180)
 		(fields_autoplaced yes)
 		(effects
@@
 		)
 		(property "Intersheetrefs" "${INTERSHEET_REFS}"
-			(at 26.89 144.78 0)
+			(at 26.89 152.4 0)
 			(effects
 				(font
@@
 	(global_label "IN2"
 		(shape input)
-		(at 33.02 149.86 180)
+		(at 33.02 144.78 180)
 		(fields_autoplaced yes)
 		(effects
@@
 		)
 		(property "Intersheetrefs" "${INTERSHEET_REFS}"
-			(at 26.89 149.86 0)
+			(at 26.89 144.78 0)
 			(effects
 				(font
@@
 	(global_label "ADC_SCL"
 		(shape input)
-		(at 29.21 96.52 180)
+		(at 29.21 88.9 180)
 		(fields_autoplaced yes)
 		(effects
@@
 		)
 		(property "Intersheetrefs" "${INTERSHEET_REFS}"
-			(at 18.121 96.52 0)
+			(at 18.121 88.9 0)
 			(effects
 				(font
@@
 	(global_label "EX+"
 		(shape input)
-		(at 107.95 177.8 180)
+		(at 107.95 170.18 180)
 		(fields_autoplaced yes)
 		(effects
@@
 		)
 		(property "Intersheetrefs" "${INTERSHEET_REFS}"
-			(at 101.0339 177.8 0)
+			(at 101.0339 170.18 0)
 			(effects
 				(font
@@
 	(global_label "IN0"
 		(shape input)
-		(at 114.3 189.23 270)
+		(at 114.3 181.61 270)
 		(fields_autoplaced yes)
 		(effects
@@
 		)
 		(property "Intersheetrefs" "${INTERSHEET_REFS}"
-			(at 114.3 195.36 90)
+			(at 114.3 187.74 90)
 			(effects
 				(font
@@
 	(global_label "EX-"
 		(shape input)
-		(at 144.78 175.26 180)
+		(at 144.78 172.72 180)
 		(fields_autoplaced yes)
 		(effects
@@
 		)
 		(property "Intersheetrefs" "${INTERSHEET_REFS}"
-			(at 137.8639 175.26 0)
+			(at 137.8639 172.72 0)
 			(effects
 				(font
@@
 	(global_label "IN2"
 		(shape input)
-		(at 144.78 170.18 180)
+		(at 144.78 177.8 180)
 		(fields_autoplaced yes)
 		(effects
@@
 		)
 		(property "Intersheetrefs" "${INTERSHEET_REFS}"
-			(at 138.65 170.18 0)
+			(at 138.65 177.8 0)
 			(effects
 				(font
@@
 	(global_label "IN3"
 		(shape input)
-		(at 144.78 172.72 180)
+		(at 144.78 175.26 180)
 		(fields_autoplaced yes)
 		(effects
@@
 		)
 		(property "Intersheetrefs" "${INTERSHEET_REFS}"
-			(at 138.65 172.72 0)
+			(at 138.65 175.26 0)
 			(effects
 				(font
@@
 	(global_label "IN1"
 		(shape input)
-		(at 130.81 189.23 270)
+		(at 130.81 181.61 270)
 		(fields_autoplaced yes)
 		(effects
@@
 		)
 		(property "Intersheetrefs" "${INTERSHEET_REFS}"
-			(at 130.81 195.36 90)
+			(at 130.81 187.74 90)
 			(effects
 				(font
@@
 	(global_label "IN3"
 		(shape input)
-		(at 33.02 152.4 180)
+		(at 33.02 147.32 180)
 		(fields_autoplaced yes)
 		(effects
@@
 		)
 		(property "Intersheetrefs" "${INTERSHEET_REFS}"
-			(at 26.89 152.4 0)
+			(at 26.89 147.32 0)
 			(effects
 				(font
@@
 	(global_label "ADC_SDA"
 		(shape input)
-		(at 29.21 93.98 180)
+		(at 29.21 91.44 180)
 		(fields_autoplaced yes)
 		(effects
@@
 		)
 		(property "Intersheetrefs" "${INTERSHEET_REFS}"
-			(at 18.0605 93.98 0)
+			(at 18.0605 91.44 0)
 			(effects
 				(font
@@
 	(global_label "IN1"
 		(shape input)
-		(at 33.02 147.32 180)
+		(at 33.02 149.86 180)
 		(fields_autoplaced yes)
 		(effects
@@
 		)
 		(property "Intersheetrefs" "${INTERSHEET_REFS}"
-			(at 26.89 147.32 0)
+			(at 26.89 149.86 0)
 			(effects
 				(font
@@
 	(symbol
 		(lib_id "Isolator:PC817")
-		(at 191.77 45.72 0)
+		(at 191.77 27.94 0)
 		(unit 1)
 		(exclude_from_sim no)
@@
 		(fields_autoplaced yes)
 		(property "Reference" "U5"
-			(at 191.77 36.83 0)
+			(at 191.77 19.05 0)
 			(effects
 				(font
@@
 		)
 		(property "Value" "PC817"
-			(at 191.77 39.37 0)
+			(at 191.77 21.59 0)
 			(effects
 				(font
@@
 		)
 		(property "Footprint" "Package_DIP:DIP-4_W7.62mm"
-			(at 186.69 50.8 0)
+			(at 186.69 33.02 0)
 			(effects
 				(font
@@
 		)
 		(property "Datasheet" "http://www.soselectronic.cz/a_info/resource/d/pc817.pdf"
-			(at 191.77 45.72 0)
+			(at 191.77 27.94 0)
 			(effects
 				(font
@@
 		)
 		(property "Description" "DC Optocoupler, Vce 35V, CTR 50-300%, DIP-4"
-			(at 191.77 45.72 0)
+			(at 191.77 27.94 0)
 			(effects
 				(font
@@
 	)
 	(symbol
-		(lib_id "power:+3.3V")
-		(at 29.21 71.12 90)
-		(unit 1)
-		(exclude_from_sim no)
-		(in_bom yes)
-		(on_board yes)
-		(dnp no)
-		(fields_autoplaced yes)
-		(property "Reference" "#PWR037"
-			(at 33.02 71.12 0)
-			(effects
-				(font
-					(size 1.27 1.27)
-				)
-				(hide yes)
-			)
-		)
-		(property "Value" "+3.3V"
-			(at 25.4 71.1199 90)
-			(effects
-				(font
-					(size 1.27 1.27)
-				)
-				(justify left)
-			)
-		)
-		(property "Footprint" ""
-			(at 29.21 71.12 0)
-			(effects
-				(font
-					(size 1.27 1.27)
-				)
-				(hide yes)
-			)
-		)
-		(property "Datasheet" ""
-			(at 29.21 71.12 0)
-			(effects
-				(font
-					(size 1.27 1.27)
-				)
-				(hide yes)
-			)
-		)
-		(property "Description" "Power symbol creates a global label with name \"+3.3V\""
-			(at 29.21 71.12 0)
-			(effects
-				(font
-					(size 1.27 1.27)
-				)
-				(hide yes)
-			)
-		)
-		(pin "1"
-		)
-		(instances
-			(project "v0.2.1"
-				(path "/f5ecb7fa-5db2-4074-ab55-2fe6f1a25df0"
-					(reference "#PWR037")
-					(unit 1)
-				)
-			)
-		)
-	)
-	(symbol
 		(lib_id "power:GNDD")
 		(at 85.09 93.98 90)
@@
 	(symbol
 		(lib_id "Device:R_Small")
-		(at 121.92 177.8 270)
+		(at 121.92 170.18 270)
 		(unit 1)
 		(exclude_from_sim no)
@@
 		(fields_autoplaced yes)
 		(property "Reference" "R9"
-			(at 121.92 172.72 90)
+			(at 121.92 165.1 90)
 			(effects
 				(font
@@
 		)
 		(property "Value" "R_Small"
-			(at 121.92 175.26 90)
+			(at 121.92 167.64 90)
 			(effects
 				(font
@@
 		)
 		(property "Footprint" "Resistor_THT:R_Axial_DIN0204_L3.6mm_D1.6mm_P7.62mm_Horizontal"
-			(at 121.92 177.8 0)
+			(at 121.92 170.18 0)
 			(effects
 				(font
@@
 		)
 		(property "Datasheet" "~"
-			(at 121.92 177.8 0)
+			(at 121.92 170.18 0)
 			(effects
 				(font
@@
 		)
 		(property "Description" "Resistor, small symbol"
-			(at 121.92 177.8 0)
+			(at 121.92 170.18 0)
 			(effects
 				(font
@@
 	(symbol
 		(lib_id "Isolator:PC817")
-		(at 191.77 27.94 0)
+		(at 191.77 45.72 0)
 		(unit 1)
 		(exclude_from_sim no)
@@
 		(fields_autoplaced yes)
 		(property "Reference" "U3"
-			(at 191.77 19.05 0)
+			(at 191.77 36.83 0)
 			(effects
 				(font
@@
 		)
 		(property "Value" "PC817"
-			(at 191.77 21.59 0)
+			(at 191.77 39.37 0)
 			(effects
 				(font
@@
 		)
 		(property "Footprint" "Package_DIP:DIP-4_W7.62mm"
-			(at 186.69 33.02 0)
+			(at 186.69 50.8 0)
 			(effects
 				(font
@@
 		)
 		(property "Datasheet" "http://www.soselectronic.cz/a_info/resource/d/pc817.pdf"
-			(at 191.77 27.94 0)
+			(at 191.77 45.72 0)
 			(effects
 				(font
@@
 		)
 		(property "Description" "DC Optocoupler, Vce 35V, CTR 50-300%, DIP-4"
-			(at 191.77 27.94 0)
+			(at 191.77 45.72 0)
 			(effects
 				(font
