File: DAQ_design/v0.2.1/CAD/v0.2.1/v0.2.1.kicad_pcb (KiCad board)
At the start: 2 copper layers, 33 parts, among them J1 Screw_Terminal_01x04, Q1 BC549, Q2 IRF9540N, Q3 IRF540N, Q4 BC549, Q5 IRF540N, Q6 IRF9540N, U1 Teensy4.0, U2 SFH617A-1X001, U3 SFH617A-1X001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

Commit message: more cad
Parts:
- removed FB1, FB2: MMZ2012Y152B, Inductor_SMD:L_Ferrocore_DLG-0302
- removed Q1, Q4: BC549, Package_TO_SOT_THT:TO-92_Inline_Wide
- removed Q2, Q6: IRF9540N, Package_TO_SOT_THT:TO-220-3_Vertical
- removed Q3, Q5: IRF540N, Package_TO_SOT_THT:TO-220-3_Vertical
- added C2: 0.1uf, Capacitor_SMD:C_1206_3216Metric, F.Cu at (175.6, 76.6)
- added R12: 10k, Resistor_SMD:R_1206_3216Metric, F.Cu at (136.1, 79.3)
- added R13: 10k, Resistor_SMD:R_1206_3216Metric, F.Cu at (129.1, 91.3)
- added S1: DS01C-254-L-09BE, dip-switch:SW_DS01C-254-L-09BE, F.Cu at (168.1, 124.8)
- added U5: PC817, Package_DIP:DIP-4_W7.62mm, F.Cu at (152.7, 96.8)
- added U6: PC817, Package_DIP:DIP-4_W7.62mm, F.Cu at (159.7, 96.6)
- C1: value 1uF -> 1uf
- R10, R11: value R_Small -> 10k
- R3, R5: value 1k -> 470
- R4: value 10k -> 470
- U2: value SFH617A-1X001 -> L293D; footprint Package_DIP:DIP-4_W7.62mm -> Package_DIP:DIP-16_W7.62mm
- U3: value SFH617A-1X001 -> PC817
- moved J1 95.7 mm to (142.8, 54.0), turned to 0 degrees
- moved 5V1 80.4 mm to (190.0, 116.0), turned to 90 degrees
- moved D1 71.8 mm to (140.6, 69.6)
- moved D3 63.9 mm to (147.4, 73.0), turned to 180 degrees
- moved D4 62.3 mm to (147.4, 69.6), turned to 180 degrees
- moved D2 59.2 mm to (140.6, 73.0)
- moved D5 55.2 mm to (152.4, 127.6), turned to -90 degrees
- moved R9 54.7 mm to (173.5, 59.1), turned to -90 degrees
- moved R2 54.3 mm to (120.1, 83.8), turned to 90 degrees
- moved U4 51.3 mm to (130.8, 76.0), turned to 180 degrees
- moved D6 50.8 mm to (149.0, 127.6), turned to -90 degrees
- moved R1 49.3 mm to (124.1, 83.8), turned to 90 degrees
- moved C1 48.9 mm to (131.1, 80.3), turned to 180 degrees
- moved R7 47.5 mm to (152.3, 121.1), turned to -90 degrees
- moved U2 42.8 mm to (179.7, 66.0), turned to -90 degrees
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Connections:
- A1 pad 6: GND -> GNDD
- C1 pad 1: Net-(U4-VDD) -> GNDD
- C1 pad 2: Net-(U4-GND) -> VDD
- D1 pad 2: GND -> GNDD
- D2 pad 2: GND -> GNDD
- D3 pad 2: GND -> GNDD
- D4 pad 2: GND -> GNDD
- J1 pad 3: IN3 -> EX-
- J1 pad 4: EX- -> IN3
- R10 pad 1: Net-(R10-Pad1) -> VPP
- R10 pad 2: LOGIC1 -> OPT2
- R11 pad 1: Net-(R11-Pad1) -> VPP
- R11 pad 2: LOGIC2 -> OPTEN
- R3 pad 1: Net-(Q1-B) -> Net-(R3-Pad1)
- R3 pad 2: OPT1 -> GNDD
- R4 pad 1: VPP -> Net-(R4-Pad1)
- R4 pad 2: Net-(Q1-C) -> GNDD
- R5 pad 2: OPT2 -> GNDD
- R6 pad 2: Net-(Q4-C) -> OPT1
- R7 pad 1: GND -> GNDD
- R8 pad 1: GND -> GNDD
- U1 pad 1: GND -> GNDD
- U1 pad 17: GND -> GNDD
- U1 pad 32: GND -> GNDD
- U1 pad 33: unconnected-(U1-VIN-Pad33) -> VDD
- U1 pad 4: LEDPOW -> EN
- U1 pad 5: LEDACT -> LEDPOW
- U1 pad 6: unconnected-(U1-4_BCLK2-Pad6) -> LEDACT
- U2 pad 1: Net-(R10-Pad1) -> OPTEN
- U2 pad 2: GND -> OPT1
- U2 pad 3: GND -> EX+
- U2 pad 4: OPT1 -> GND
- U3 pad 1: Net-(R11-Pad1) -> LOGIC1
- U3 pad 2: GND -> Net-(R3-Pad1)
- U3 pad 4: OPT2 -> OPT1
- U4 pad 1: GND -> Net-(U4-ADDR)
- U4 pad 2: unconnected-(U4-ALERT/RDY-Pad2) -> Net-(U4-ALERT/RDY)
- U4 pad 3: Net-(U4-GND) -> GNDD
- U4 pad 8: Net-(U4-VDD) -> VDD
Routing:
- net VPP: track 130.9 -> 0.00 mm, vias 1 -> 0
- net ADC_SDA: track 105.3 -> 0.00 mm
- net EX+: track 102.4 -> 0.00 mm
- net ADC_SCL: track 98.8 -> 0.00 mm
- net IN3: track 92.8 -> 0.00 mm
- net IN0: track 89.3 -> 0.00 mm
- net IN1: track 84.4 -> 0.00 mm, vias 2 -> 0
- net OPT1: track 70.3 -> 0.00 mm
- net LEDPOW: track 63.3 -> 0.00 mm
- net Net-(Q4-C): track 50.9 -> 0.00 mm, vias 1 -> 0
- net LEDACT: track 50.4 -> 0.00 mm, vias 1 -> 0
- net LOGIC2: track 47.7 -> 0.00 mm
- net OPT2: track 46.3 -> 0.00 mm
- net +3.3V: track 39.7 -> 0.00 mm
- net SDCLK: track 37.5 -> 0.00 mm
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Other:
- board outline added: 100 x 80 mm

Commit message: power planes
Parts:
- D1, D2, D3, D4: footprint Diode_SMD:D_1206_3216Metric -> Diode_THT:D_DO-35_SOD27_P7.62mm_Horizontal
- D5: footprint LED_SMD:LED_1206_3216Metric -> LED_THT:LED_D5.0mm_Horizontal_O1.27mm_Z3.0mm_IRGrey
- D6: footprint LED_SMD:LED_1206_3216Metric -> LED_THT:LED_D5.0mm_Horizontal_O1.27mm_Z3.0mm
- R9: footprint Resistor_SMD:R_1206_3216Metric -> Resistor_THT:R_Axial_DIN0204_L3.6mm_D1.6mm_P7.62mm_Horizontal
- moved D6 40.3 mm to (187.5, 139.7)
- moved D5 40.0 mm to (187.5, 146.7)
- moved D1 37.6 mm to (178.0, 65.8), turned to 90 degrees
- moved S1 32.1 mm to (136.0, 124.8)
- moved R7 25.3 mm to (177.6, 121.1)
- moved R8 25.3 mm to (174.3, 121.1)
- moved A1 25.3 mm to (166.3, 113.3)
- moved D2 14.1 mm to (152.8, 66.0), turned to 180 degrees
- moved D3 13.8 mm to (142.8, 60.0)
- moved R13 11.9 mm to (135.0, 81.0), turned to 90 degrees
- moved C1 7.87 mm to (124.5, 76.0), turned to 0 degrees
- moved C2 7.24 mm to (182.0, 80.0), turned to 180 degrees
- moved D4 6.62 mm to (147.8, 63.0)
- moved R2 6.20 mm to (124.0, 79.0), turned to 0 degrees
- moved R12 4.46 mm to (132.0, 81.0)
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Connections:
- D1 pad 1: IN0 -> EX+
- D3 pad 1: EX+ -> IN2
- J1 pad 1: IN0 -> IN2
- J1 pad 2: IN1 -> IN3
- J1 pad 4: IN3 -> IN1
- R9 pad 1: IN3 -> IN1
- U4 pad 4: IN0 -> EX+
- U4 pad 6: EX+ -> IN2
Routing:
- added copper zone on F.Cu, net GNDD

Commit message: 74hc165
Parts:
- added C3: 0.1uf, Capacitor_SMD:C_1206_3216Metric, F.Cu at (77.4, 140.8)
- added R14: 10k, Resistor_SMD:R_1206_3216Metric, F.Cu at (124.0, 117.5)
- added R15: 10k, Resistor_SMD:R_1206_3216Metric, F.Cu at (127.3, 117.5)
- added R16: 10k, Resistor_SMD:R_1206_3216Metric, F.Cu at (130.6, 117.5)
- added R17: 10k, Resistor_SMD:R_1206_3216Metric, F.Cu at (133.9, 117.5)
- added R18: 10k, Resistor_SMD:R_1206_3216Metric, F.Cu at (137.2, 117.5)
- added R19: 10k, Resistor_SMD:R_1206_3216Metric, F.Cu at (140.4, 117.5)
- added R20: 10k, Resistor_SMD:R_1206_3216Metric, F.Cu at (143.7, 117.5)
- added R21: 10k, Resistor_SMD:R_1206_3216Metric, F.Cu at (147.0, 117.5)
- added R22: 10k, Resistor_SMD:R_1206_3216Metric, F.Cu at (150.3, 117.5)
- added U7: 74HC165, Package_DIP:DIP-16_W7.62mm, F.Cu at (141.9, 139.2)
- D5: footprint LED_THT:LED_D5.0mm_Horizontal_O1.27mm_Z3.0mm_IRGrey -> LED_SMD:LED_1206_3216Metric_Pad1.42x1.75mm_HandSolder
- D6: footprint LED_THT:LED_D5.0mm_Horizontal_O1.27mm_Z3.0mm -> LED_SMD:LED_1206_3216Metric_Pad1.42x1.75mm_HandSolder
- S1: value DS01C-254-L-09BE -> DS03-254-10BE; footprint dip-switch:SW_DS01C-254-L-09BE -> dip-switch:SW_DS03-254-10BE
- moved S1 2.08 mm to (136.1, 122.7)
- moved A1 1.73 mm to (168.1, 113.3)
Connections:
- C1 pad 2: VDD -> SW1
- R1 pad 1: VDD -> SW1
- R13 pad 1: VDD -> SW1
- R2 pad 1: VDD -> SW1
- S1 pad 1A: unconnected-(S1-Pad1A) -> SW1
- S1 pad 1B: unconnected-(S1-Pad1B) -> Net-(R14-Pad2)
- S1 pad 2A: unconnected-(S1-Pad2A) -> SW1
- S1 pad 2B: unconnected-(S1-Pad2B) -> Net-(R15-Pad2)
- S1 pad 3A: unconnected-(S1-Pad3A) -> SW1
- S1 pad 3B: unconnected-(S1-Pad3B) -> Net-(R16-Pad2)
- S1 pad 4A: unconnected-(S1-Pad4A) -> SW1
- S1 pad 4B: unconnected-(S1-Pad4B) -> Net-(R17-Pad2)
- S1 pad 5A: unconnected-(S1-Pad5A) -> SW1
- S1 pad 5B: unconnected-(S1-Pad5B) -> Net-(R18-Pad2)
- S1 pad 6A: unconnected-(S1-Pad6A) -> SW1
- S1 pad 6B: unconnected-(S1-Pad6B) -> Net-(R19-Pad2)
- S1 pad 7A: unconnected-(S1-Pad7A) -> SW1
- S1 pad 7B: unconnected-(S1-Pad7B) -> Net-(R20-Pad2)
- S1 pad 8A: unconnected-(S1-Pad8A) -> SW1
- S1 pad 8B: unconnected-(S1-Pad8B) -> Net-(R21-Pad2)
- S1 pad 9B: unconnected-(S1-Pad9B) -> Net-(R22-Pad2)
- U1 pad 10: unconnected-(U1-8_TX2_IN1-Pad10) -> LOGIC1
- U1 pad 11: unconnected-(U1-9_OUT1C-Pad11) -> LOGIC2
- U1 pad 16: unconnected-(U1-3V3-Pad16) -> +3.3V
- U1 pad 2: LOGIC1 -> unconnected-(U1-0_RX1_CRX2_CS1-Pad2)
- U1 pad 3: LOGIC2 -> unconnected-(U1-1_TX1_CTX2_MISO1-Pad3)
- U1 pad 33: VDD -> SW1
- U1 pad 7: unconnected-(U1-5_IN2-Pad7) -> DIPDAT
- U1 pad 8: unconnected-(U1-6_OUT1D-Pad8) -> DIPLAT
- U1 pad 9: unconnected-(U1-7_RX2_OUT1A-Pad9) -> DIPCP
- U4 pad 8: VDD -> SW1

Commit message: routing progress
Parts:
- removed R22: 10k, Resistor_SMD:R_1206_3216Metric
- R14, R15, R16, R17, R18, R19, R20, R21: footprint Resistor_SMD:R_1206_3216Metric -> Resistor_SMD:R_0805_2012Metric
- moved C3 68.6 mm to (144.5, 155.0)
- moved U7 41.9 mm to (133.4, 98.2), turned to 0 degrees
- moved R18 16.1 mm to (144.4, 103.1), turned to 180 degrees
- moved R17 14.9 mm to (130.1, 103.0), turned to 0 degrees
- moved R19 12.1 mm to (144.4, 106.0), turned to 180 degrees
- moved R16 11.5 mm to (130.1, 106.0), turned to 0 degrees
- moved R15 8.91 mm to (130.1, 109.0), turned to 0 degrees
- moved R20 8.49 mm to (144.4, 109.0), turned to 180 degrees
- moved R14 8.11 mm to (130.0, 112.0), turned to 0 degrees
- moved R21 6.06 mm to (144.4, 112.0), turned to 180 degrees
- moved R10 3.74 mm to (156.7, 83.3)
- moved R11 3.74 mm to (163.7, 83.3)
- moved R3 3.74 mm to (152.0, 103.3)
- moved R4 3.74 mm to (159.0, 103.3)
- moved R5 3.74 mm to (166.0, 103.3)
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Connections:
- C1 pad 2: SW1 -> VDD
- C3 pad 2: SW1 -> VDD
- R1 pad 1: SW1 -> VDD
- R13 pad 1: SW1 -> VDD
- R14 pad 2: Net-(R14-Pad2) -> SW8
- R15 pad 2: Net-(R15-Pad2) -> SW7
- R16 pad 2: Net-(R16-Pad2) -> SW6
- R17 pad 2: Net-(R17-Pad2) -> SW5
- R18 pad 2: Net-(R18-Pad2) -> SW4
- R19 pad 2: Net-(R19-Pad2) -> SW3
- R2 pad 1: SW1 -> VDD
- R20 pad 2: Net-(R20-Pad2) -> SW2
- R21 pad 2: Net-(R21-Pad2) -> SW1
- S1 pad 1A: SW1 -> VDD
- S1 pad 1B: Net-(R14-Pad2) -> SW8
- S1 pad 2A: SW1 -> VDD
- S1 pad 2B: Net-(R15-Pad2) -> SW7
- S1 pad 3A: SW1 -> VDD
- S1 pad 3B: Net-(R16-Pad2) -> SW6
- S1 pad 4A: SW1 -> VDD
- S1 pad 4B: Net-(R17-Pad2) -> SW5
- S1 pad 5A: SW1 -> VDD
- S1 pad 5B: Net-(R18-Pad2) -> SW4
- S1 pad 6A: SW1 -> VDD
- S1 pad 6B: Net-(R19-Pad2) -> SW3
- S1 pad 7A: SW1 -> VDD
- S1 pad 7B: Net-(R20-Pad2) -> SW2
- S1 pad 8A: SW1 -> VDD
- S1 pad 8B: Net-(R21-Pad2) -> SW1
- S1 pad 9B: Net-(R22-Pad2) -> unconnected-(S1-Pad9B)
- U1 pad 33: SW1 -> VDD
- U4 pad 8: SW1 -> VDD
- U7 pad 12: SW1 -> SW2
- U7 pad 13: SW1 -> SW3
- U7 pad 14: SW1 -> SW4
- U7 pad 16: SW1 -> VDD
- U7 pad 3: SW1 -> SW5
- U7 pad 4: SW1 -> SW6
- U7 pad 5: SW1 -> SW7
- U7 pad 6: SW1 -> SW8
Routing:
- net SW5: track 0.00 -> 23.7 mm
- net SW4: track 0.00 -> 23.5 mm
- net SW6: track 0.00 -> 21.5 mm
- net SW3: track 0.00 -> 21.3 mm
- net VDD: track 0.00 -> 20.5 mm
- net SW7: track 0.00 -> 19.5 mm
- net SW2: track 0.00 -> 19.3 mm
- net SW1: track 0.00 -> 19.1 mm
- net SW8: track 0.00 -> 18.4 mm
- net Net-(R5-Pad1): track 0.00 -> 5.28 mm
- net Net-(R3-Pad1): track 0.00 -> 5.20 mm
- net Net-(R4-Pad1): track 0.00 -> 5.00 mm
- net Net-(U4-ALERT/RDY): track 0.00 -> 4.32 mm
- net OPT2: track 0.00 -> 4.29 mm
- net OPTEN: track 0.00 -> 4.09 mm
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
Commit message: update v0.2.1 cad
Parts:
- removed C1: 1uf, Capacitor_SMD:C_1206_3216Metric
- removed D1: zener1, Diode_THT:D_DO-35_SOD27_P7.62mm_Horizontal
- removed D2: zener2, Diode_THT:D_DO-35_SOD27_P7.62mm_Horizontal
- removed D3: zener3, Diode_THT:D_DO-35_SOD27_P7.62mm_Horizontal
- removed D4: zener4, Diode_THT:D_DO-35_SOD27_P7.62mm_Horizontal
- removed R1, R12, R13: 10k, Resistor_SMD:R_1206_3216Metric
- removed R2: 10K, Resistor_SMD:R_1206_3216Metric
- removed S1: DS03-254-10BE, dip-switch:SW_DS03-254-10BE
- removed U4: ADS1115IDGS, Package_SO:TSSOP-10_3x3mm_P0.5mm
- added A2: ADS1115_ADC_Module, Charleslabs_Parts:ADC1115_ADC_Module, F.Cu at (106.6, 57.2)
- added D10: zener4, Diode_THT:D_DO-35_SOD27_P7.62mm_Horizontal, F.Cu at (116.4, 67.5)
- added D7: zener1, Diode_THT:D_DO-35_SOD27_P7.62mm_Horizontal, F.Cu at (116.4, 56.9)
- added D8: zener2, Diode_THT:D_DO-35_SOD27_P7.62mm_Horizontal, F.Cu at (116.4, 60.4)
- added D9: zener3, Diode_THT:D_DO-35_SOD27_P7.62mm_Horizontal, F.Cu at (116.4, 64.0)
- added R22: 10k, Resistor_SMD:R_1206_3216Metric, F.Cu at (117.6, 70.9)
- added S2: 76PSB08ST, 8-pos-dip-switch-foot:76PSB08ST, F.Cu at (128.5, 128.1)
- moved R14 2.83 mm to (128.0, 110.0)
- moved R15 2.83 mm to (128.1, 107.0)
- moved R16 2.83 mm to (128.1, 104.0)
- moved R17 2.83 mm to (128.1, 101.0)
- moved R18 2.83 mm to (142.4, 101.1)
- moved R19 2.83 mm to (142.4, 104.0)
- moved R20 2.83 mm to (142.4, 107.0)
- moved R21 2.83 mm to (142.4, 110.0)
- moved U7 2.83 mm to (131.4, 96.2)
Routing:
- net VDD: track 20.5 -> 0.00 mm
- net SW5: track 23.7 -> 5.91 mm
- net SW4: track 23.5 -> 5.88 mm
- net SW6: track 21.5 -> 5.34 mm
- net SW3: track 21.3 -> 5.34 mm
- net SW7: track 19.5 -> 5.01 mm
- net SW1: track 19.1 -> 4.69 mm
- net SW2: track 19.3 -> 5.01 mm
- net SW8: track 18.4 -> 4.78 mm
- net Net-(U4-ALERT/RDY): track 4.32 -> 0.00 mm
- net Net-(U4-ADDR): track 2.95 -> 0.00 mm
- net GNDD: track 2.02 -> 0.00 mm, vias 1 -> 0

Commit message: i am a moron
Parts:
- D10, D7, D8, D9: footprint Diode_THT:D_DO-35_SOD27_P7.62mm_Horizontal -> Diode_SMD:D_1206_3216Metric_Pad1.42x1.75mm_HandSolder
- R22: footprint Resistor_SMD:R_1206_3216Metric -> Resistor_SMD:R_0805_2012Metric
- moved A2 39.2 mm to (143.6, 70.0), turned to -90 degrees
- moved C3 30.2 mm to (151.0, 125.5), turned to -90 degrees
- moved D5 21.7 mm to (178.5, 127.0)
- moved D6 17.5 mm to (175.5, 127.0)
- moved R9 17.0 mm to (158.0, 59.2)
- moved R22 16.7 mm to (133.6, 66.0), turned to 90 degrees
- moved D7 15.4 mm to (129.5, 65.0), turned to 90 degrees
- moved D8 11.1 mm to (126.5, 65.0), turned to 90 degrees
- moved D9 7.20 mm to (123.5, 65.0), turned to 90 degrees
- moved D10 4.82 mm to (120.5, 65.0), turned to -90 degrees
- moved A1 3.23 mm to (168.1, 113.3)
- moved R3 2.27 mm to (154.3, 103.5)
- moved R4 2.27 mm to (161.3, 103.5)
- moved U3 2.27 mm to (151.7, 96.8)
- moved U5 2.27 mm to (158.7, 97.0)
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
Commit message: figuring out battery
Parts:
- removed 5V1: Barrel_Jack, Connector_BarrelJack:BarrelJack_Horizontal
- moved D5 104.2 mm to (97.0, 62.0), turned to 180 degrees
- moved D6 103.9 mm to (97.0, 59.0), turned to 180 degrees
- moved R7 96.6 mm to (102.5, 62.0), turned to 180 degrees
- moved R8 96.1 mm to (102.5, 59.0), turned to 180 degrees
- moved J1 72.9 mm to (209.0, 84.7), turned to -90 degrees
- moved D10 70.4 mm to (190.4, 73.5), turned to 90 degrees
- moved S2 67.2 mm to (96.3, 69.1), turned to -90 degrees
- moved D9 64.4 mm to (187.4, 73.5), turned to -90 degrees
- moved R9 61.2 mm to (203.8, 99.8), turned to 180 degrees
- moved D8 58.5 mm to (184.4, 73.5), turned to -90 degrees
- moved A1 55.4 mm to (113.2, 106.3), turned to 180 degrees
- moved D7 52.6 mm to (181.4, 73.5), turned to -90 degrees
- moved C3 46.6 mm to (127.8, 85.1), turned to 90 degrees
- moved R22 44.2 mm to (177.3, 72.5), turned to -90 degrees
- moved R14 42.7 mm to (114.4, 70.1), turned to -90 degrees
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Routing:
- removed copper zone on B.Cu, net GND
- removed copper zone on F.Cu, net GNDD
Other:
- board size 100 x 80 mm -> 119 x 75 mm

Commit message: bad traces
Parts:
- moved D6 65.3 mm to (114.0, 122.0), turned to 0 degrees
- moved R8 63.2 mm to (107.5, 122.0), turned to 0 degrees
- moved D5 59.1 mm to (114.0, 118.6), turned to 0 degrees
- moved R7 56.9 mm to (107.5, 118.7), turned to 0 degrees
- moved D10 43.7 mm to (151.4, 93.3)
- moved D9 38.6 mm to (151.5, 87.8), turned to 90 degrees
- moved D8 34.0 mm to (151.5, 82.3), turned to 90 degrees
- moved C3 31.9 mm to (141.3, 56.2)
- moved D7 30.0 mm to (151.5, 76.8), turned to 90 degrees
- moved U3 19.2 mm to (152.9, 103.8)
- moved R3 19.0 mm to (146.5, 106.3)
- moved R4 19.0 mm to (146.5, 113.3)
- moved U5 18.8 mm to (152.9, 110.5)
- moved U7 18.8 mm to (130.5, 54.8), turned to 0 degrees
- moved U6 18.6 mm to (152.9, 117.2)
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Routing:
- net VDD: track 0.00 -> 103.5 mm
- net EX+: track 0.00 -> 92.4 mm
- net DIPLAT: track 0.00 -> 80.6 mm, vias 0 -> 1
- net DIPCP: track 0.00 -> 74.7 mm
- net IN2: track 0.00 -> 74.0 mm, vias 0 -> 1
- net IN3: track 0.00 -> 71.4 mm
- net IN1: track 0.00 -> 67.0 mm
- net ADC_SCL: track 0.00 -> 61.8 mm
- net VPP: track 0.00 -> 61.1 mm
- net DIPDAT: track 0.00 -> 57.1 mm
- net EX-: track 0.00 -> 51.6 mm
- net +3.3V: track 0.00 -> 44.6 mm
- net SDMISO: track 0.00 -> 43.7 mm, vias 0 -> 1
- net ADC_SDA: track 0.00 -> 43.3 mm
- net EN: track 0.00 -> 43.0 mm
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- added copper zone on B.Cu, net GND
- added copper zone on F.Cu, net GND
- added copper zone on B.Cu, net GNDD
- added copper zone on F.Cu, net GNDD
