File: DAQ_design/v0.2.1/CAD/v0.2.1/v0.2.1.kicad_pcb (KiCad board)
At the start: 2 copper layers, 119 x 75 mm, 36 parts, among them J1 Screw_Terminal_01x04, U1 Teensy4.0, U2 L293D, U3 PC817, U5 PC817, U6 PC817, U7 74HC165

Commit message: sync
Parts:
- moved C2 26.4 mm to (173.9, 118.7), turned to 90 degrees
- moved U2 22.6 mm to (184.5, 116.9), turned to 180 degrees
- moved A1 2.00 mm to (122.0, 93.5)
- moved U1 0.70 mm to (122.0, 106.6)
Routing:
- net VDD: track 103.5 -> 0.00 mm
- net EX+: track 92.4 -> 0.00 mm
- net DIPLAT: track 80.6 -> 0.00 mm, vias 1 -> 0
- net DIPCP: track 74.7 -> 0.00 mm
- net IN2: track 74.0 -> 0.00 mm, vias 1 -> 0
- net IN3: track 71.4 -> 0.00 mm
- net IN1: track 67.0 -> 0.00 mm
- net ADC_SCL: track 61.8 -> 0.00 mm
- net VPP: track 61.1 -> 0.00 mm
- net DIPDAT: track 57.1 -> 0.00 mm
- net EX-: track 51.6 -> 0.00 mm
- net +3.3V: track 44.6 -> 0.00 mm
- net SDMISO: track 43.7 -> 0.00 mm, vias 1 -> 0
- net ADC_SDA: track 43.3 -> 0.00 mm
- net EN: track 43.0 -> 0.00 mm
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
Commit message: resync
Parts:
- moved R9 48.0 mm to (185.0, 123.7), turned to 180 degrees
- moved C3 30.2 mm to (128.8, 83.7), turned to 0 degrees
- moved D6 27.2 mm to (90.0, 134.8), turned to 180 degrees
- moved D5 26.9 mm to (89.9, 130.5), turned to 180 degrees
- moved R3 25.6 mm to (128.9, 124.9)
- moved R6 25.5 mm to (149.2, 120.8)
- moved D7 23.9 mm to (133.9, 92.9), turned to 180 degrees
- moved D8 22.1 mm to (134.0, 95.7), turned to 180 degrees
- moved R11 21.6 mm to (149.0, 127.7)
- moved R14 21.5 mm to (104.1, 68.4)
- moved U6 21.3 mm to (135.3, 129.2)
- moved R5 21.3 mm to (128.9, 131.7)
- moved U5 21.3 mm to (135.3, 122.4)
- moved A1 21.3 mm to (104.4, 105.4)
- moved A2 21.3 mm to (140.4, 78.1)
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Connections:
- A2 pad 10: IN3 -> EX+
- A2 pad 7: EX+ -> IN2
- A2 pad 8: IN1 -> IN3
- A2 pad 9: IN2 -> IN1
- D10 pad 1: IN3 -> EX+
- D7 pad 1: EX+ -> IN2
- D8 pad 1: IN1 -> IN3
- D9 pad 1: IN2 -> IN1
- J1 pad 1: IN2 -> IN1
- J1 pad 2: IN3 -> EX-
- J1 pad 3: EX- -> IN3
- J1 pad 4: IN1 -> IN2
- U1 pad 16: +3.3V -> unconnected-(U1-3V3-Pad16)
- U1 pad 23: unconnected-(U1-16_A2_RX4_SCL1-Pad23) -> ADC_SCL
- U1 pad 24: unconnected-(U1-17_A3_TX4_SDA1-Pad24) -> ADC_SDA
- U1 pad 25: ADC_SDA -> unconnected-(U1-18_A4_SDA0-Pad25)
- U1 pad 26: ADC_SCL -> unconnected-(U1-19_A5_SCL0-Pad26)
- U3 pad 1: LOGIC1 -> LOGIC2
- U3 pad 2: Net-(R3-Pad1) -> Net-(R4-Pad1)
- U3 pad 4: OPT1 -> OPT2
- U5 pad 1: LOGIC2 -> LOGIC1
- U5 pad 2: Net-(R4-Pad1) -> Net-(R3-Pad1)
- U5 pad 4: OPT2 -> OPT1
Routing:
- net IN1: track 0.00 -> 90.5 mm
- net EX+: track 0.00 -> 70.7 mm
- net IN3: track 0.00 -> 66.0 mm
- net IN2: track 0.00 -> 65.2 mm
- net EN: track 0.00 -> 41.0 mm
- net EX-: track 0.00 -> 38.7 mm
- net GNDD: track 0.00 -> 29.2 mm, vias 0 -> 17
- net OPT1: track 0.00 -> 25.7 mm
- net OPTEN: track 0.00 -> 25.1 mm
- net OPT2: track 0.00 -> 24.9 mm
- net LEDACT: track 0.00 -> 16.9 mm, vias 0 -> 1
- net +3.3V: track 0.00 -> 13.7 mm
- net LEDPOW: track 0.00 -> 12.5 mm, vias 0 -> 1
- net VPP: track 0.00 -> 10.6 mm, vias 0 -> 3
- net Net-(R5-Pad1): track 0.00 -> 4.92 mm
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- added copper zone on In1.Cu, net GND
- added copper zone on In1.Cu, net GNDD
- added copper zone on In2.Cu, net VDD
- added copper zone on In2.Cu, net VPP
- removed copper zone on B.Cu, net GND
- removed copper zone on B.Cu, net GNDD
- removed copper zone on F.Cu, net GNDD
Other:
- copper layers 2 -> 4

Commit message: v2 trances
Parts:
- added BT1: Battery, Connector_JST:JST_GH_SM02B-GHS-TB_1x02-1MP_P1.25mm_Horizontal, B.Cu at (197.6, 74.6)
- moved U1 19.8 mm to (104.5, 98.8)
- moved A1 18.9 mm to (104.5, 124.3)
Connections:
- U1 pad 10: LOGIC1 -> unconnected-(U1-8_TX2_IN1-Pad10)
- U1 pad 11: LOGIC2 -> unconnected-(U1-9_OUT1C-Pad11)
- U1 pad 21: unconnected-(U1-14_A0_TX3_SPDIF_OUT-Pad21) -> LOGIC1
- U1 pad 22: unconnected-(U1-15_A1_RX3_SPDIF_IN-Pad22) -> LOGIC2
- U1 pad 25: unconnected-(U1-18_A4_SDA0-Pad25) -> DIPLAT
- U1 pad 26: unconnected-(U1-19_A5_SCL0-Pad26) -> DIPCP
- U1 pad 30: unconnected-(U1-23_A9_CRX1_MCLK1-Pad30) -> DIPDAT
- U1 pad 7: DIPDAT -> unconnected-(U1-5_IN2-Pad7)
- U1 pad 8: DIPLAT -> unconnected-(U1-6_OUT1D-Pad8)
- U1 pad 9: DIPCP -> unconnected-(U1-7_RX2_OUT1A-Pad9)
Routing:
- net SDCLK: track 0.00 -> 49.7 mm
- net LOGIC1: track 0.00 -> 49.5 mm
- net LOGIC2: track 0.00 -> 40.6 mm
- net SDCS: track 0.00 -> 33.0 mm
- net ADC_SDA: track 0.00 -> 31.8 mm
- net SDMOSI: track 0.00 -> 31.5 mm
- net DIPLAT: track 0.00 -> 31.3 mm
- net DIPCP: track 0.00 -> 31.3 mm
- net ADC_SCL: track 0.00 -> 30.4 mm
- net SW4: track 0.00 -> 29.4 mm
- net SW5: track 0.00 -> 29.0 mm
- net SDMISO: track 0.00 -> 28.3 mm
- net SW3: track 0.00 -> 27.4 mm
- net SW2: track 0.00 -> 27.3 mm
- net SW6: track 0.00 -> 27.1 mm
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- added copper zone on B.Cu, net GND
- added copper zone on B.Cu, net GNDD
- added copper zone on F.Cu, net VDD
- added copper zone on F.Cu, net VPP
- removed copper zone on In1.Cu, net GND
- removed copper zone on In1.Cu, net GNDD
- removed copper zone on In2.Cu, net VDD
- removed copper zone on In2.Cu, net VPP

Commit message: bom
Parts:
- moved S2 2.75 mm to (87.5, 68.4)
Connections:
- U1 pad 17: GNDD -> unconnected-(U1-GND-Pad17)
Routing:
- net GNDD: track 46.1 -> 50.5 mm, vias 17 -> 18
- net SW7: track 26.4 -> 29.2 mm
- net SW6: track 27.1 -> 29.8 mm
- net SW5: track 29.0 -> 31.8 mm
- net SW4: track 29.4 -> 32.1 mm
- net SW3: track 27.4 -> 30.2 mm
- net SW2: track 27.3 -> 30.1 mm
- net SW1: track 25.5 -> 28.2 mm
- net SW8: track 25.2 -> 28.0 mm
Changed lines of the file:
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@@
 	(net 61 "unconnected-(U1-5_IN2-Pad7)")
 	(net 62 "unconnected-(U1-6_OUT1D-Pad8)")
+	(net 63 "unconnected-(U1-GND-Pad17)")
 	(footprint "TerminalBlock:TerminalBlock_bornier-4_P5.08mm"
 		(layer "F.Cu")
@@
 			(layers "*.Cu" "*.Mask")
 			(remove_unused_layers no)
-			(net 40 "GNDD")
+			(net 63 "unconnected-(U1-GND-Pad17)")
 			(pinfunction "GND")
 			(pintype "power_in")
@@
 	(footprint "8-pos-dip-switch-foot:76PSB08ST"
 		(layer "F.Cu")
-		(at 90.28 68.4125 -90)
+		(at 87.5325 68.41 -90)
 		(descr "76PSB08ST-3")
 		(tags "Switch")
@@
 	)
 	(segment
-		(start 103.1475 85.9125)
-		(end 97.9 85.9125)
-		(width 0.2)
-		(layer "F.Cu")
-		(net 18)
-	)
-	(segment
 		(start 116.29 79.3625)
 		(end 111.4375 79.3625)
@@
 	)
 	(segment
+		(start 95.155 85.9125)
+		(end 95.1525 85.91)
+		(width 0.3)
+		(layer "F.Cu")
+		(net 18)
+	)
+	(segment
+		(start 103.1475 85.9125)
+		(end 95.155 85.9125)
+		(width 0.3)
+		(layer "F.Cu")
+		(net 18)
+	)
+	(segment
 		(start 104.1975 86.9625)
 		(end 103.1475 85.9125)
@@
 	)
 	(segment
+		(start 118 83.6125)
+		(end 114.9 80.5125)
+		(width 0.3)
+		(layer "F.Cu")
+		(net 40)
+	)
+	(segment
 		(start 127.325 83.6925)
 		(end 127.325 80.7875)
@@
 	)
 	(segment
+		(start 118 83.7)
+		(end 118 83.6125)
+		(width 0.3)
+		(layer "F.Cu")
+		(net 40)
+	)
+	(segment
 		(start 105.0725 83.3125)
 		(end 104.9725 83.4125)
@@
 		(net 40)
 	)
+	(via
+		(at 118 83.7)
+		(size 1)
+		(drill 0.5)
+		(layers "F.Cu" "B.Cu")
+		(free yes)
+		(net 40)
+	)
 	(segment
 		(start 113.75 83.13)
@@
 	)
 	(segment
+		(start 109.8 80.292893)
+		(end 109.8 83.4)
+		(width 0.3)
+		(layer "F.Cu")
+		(net 51)
+	)
+	(segment
 		(start 103.1475 83.4125)
-		(end 97.9 83.4125)
-		(width 0.2)
+		(end 95.155 83.4125)
+		(width 0.3)
 		(layer "F.Cu")
 		(net 51)
 	)
 	(segment
-		(start 109.8 80.292893)
-		(end 109.8 83.4)
+		(start 95.155 83.4125)
+		(end 95.1525 83.41)
 		(width 0.3)
 		(layer "F.Cu")
@@
 	)
 	(segment
-		(start 103.1475 80.9125)
-		(end 97.9 80.9125)
-		(width 0.2)
-		(layer "F.Cu")
-		(net 52)
-	)
-	(segment
 		(start 104.1975 81.9625)
 		(end 103.1475 80.9125)
@@
 	)
 	(segment
+		(start 103.1475 80.9125)
+		(end 95.155 80.9125)
+		(width 0.3)
+		(layer "F.Cu")
+		(net 52)
+	)
+	(segment
 		(start 107.423287 81.9625)
 		(end 104.1975 81.9625)
@@
 	)
 	(segment
+		(start 95.155 80.9125)
+		(end 95.1525 80.91)
+		(width 0.3)
+		(layer "F.Cu")
+		(net 52)
+	)
+	(segment
+		(start 95.155 78.4125)
+		(end 95.1525 78.41)
+		(width 0.3)
+		(layer "F.Cu")
+		(net 53)
+	)
+	(segment
 		(start 108.5375 77.8625)
 		(end 107.6 78.8)
@@
 	(segment
 		(start 103.1475 78.4125)
-		(end 97.9 78.4125)
-		(width 0.2)
+		(end 95.155 78.4125)
+		(width 0.3)
 		(layer "F.Cu")
 		(net 53)
@@
 	)
 	(segment
-		(start 103.1475 75.9125)
-		(end 97.9 75.9125)
-		(width 0.2)
-		(layer "F.Cu")
-		(net 54)
-	)
-	(segment
 		(start 106.889582 74.8)
 		(end 104.26 74.8)
@@
 	)
 	(segment
+		(start 103.1475 75.9125)
+		(end 102.6125 75.9125)
+		(width 0.3)
+		(layer "F.Cu")
+		(net 54)
+	)
+	(segment
+		(start 102.61 75.91)
+		(end 95.1525 75.91)
+		(width 0.3)
+		(layer "F.Cu")
+		(net 54)
+	)
+	(segment
 		(start 107.632082 75.5425)
 		(end 106.889582 74.8)
@@
 	)
 	(segment
+		(start 102.6125 75.9125)
+		(end 102.61 75.91)
+		(width 0.3)
+		(layer "F.Cu")
+		(net 54)
+	)
+	(segment
 		(start 104.26 74.8)
 		(end 103.1475 75.9125)
@@
 	)
 	(segment
+		(start 95.155 73.4125)
+		(end 95.1525 73.41)
+		(width 0.3)
+		(layer "F.Cu")
+		(net 55)
+	)
+	(segment
 		(start 103.1475 73.4125)
-		(end 97.9 73.4125)
-		(width 0.2)
+		(end 95.155 73.4125)
+		(width 0.3)
 		(layer "F.Cu")
 		(net 55)
@@
 	)
 	(segment
+		(start 95.155 70.9125)
+		(end 95.1525 70.91)
+		(width 0.3)
+		(layer "F.Cu")
+		(net 56)
+	)
+	(segment
 		(start 109.8 71)
 		(end 108.6625 69.8625)
@@
 	(segment
 		(start 103.1475 70.9125)
-		(end 97.9 70.9125)
-		(width 0.2)
+		(end 95.155 70.9125)
+		(width 0.3)
 		(layer "F.Cu")
 		(net 56)
 	)
 	(segment
-		(start 104.37 67.2)
-		(end 103.1475 68.4225)
+		(start 95.165 68.4225)
+		(end 95.1525 68.41)
 		(width 0.3)
 		(layer "F.Cu")
@@
 	)
 	(segment
-		(start 103.1475 68.4225)
-		(end 97.91 68.4225)
-		(width 0.2)
+		(start 104.37 67.2)
+		(end 103.1475 68.4225)
+		(width 0.3)
 		(layer "F.Cu")
 		(net 57)
@@
 	)
 	(segment
-		(start 117.44 72.8925)
-		(end 116.29 74.0425)
+		(start 103.1475 68.4225)
+		(end 95.165 68.4225)
 		(width 0.3)
 		(layer "F.Cu")
@@
 	)
 	(segment
-		(start 110.4 73)
-		(end 110.4 69.8)
+		(start 117.44 72.8925)
+		(end 116.29 74.0425)
 		(width 0.3)
 		(layer "F.Cu")
@@
 	)
 	(segment
-		(start 97.91 68.4225)
-		(end 97.9 68.4125)
-		(width 0.2)
+		(start 110.4 73)
+		(end 110.4 69.8)
+		(width 0.3)
 		(layer "F.Cu")
 		(net 57)
@@
 		(min_thickness 0.25)
 		(filled_areas_thickness no)
-		(fill
+		(fill yes
 			(thermal_gap 0.5)
 			(thermal_bridge_width 0.5)
@@
 		(min_thickness 0.25)
 		(filled_areas_thickness no)
-		(fill
+		(fill yes
 			(thermal_gap 0.5)
 			(thermal_bridge_width 0.5)
@@
 		(min_thickness 0.25)
 		(filled_areas_thickness no)
-		(fill
+		(fill yes
 			(thermal_gap 0.5)
 			(thermal_bridge_width 0.5)
@@
 		(min_thickness 0.25)
 		(filled_areas_thickness no)
-		(fill
+		(fill yes
 			(thermal_gap 0.5)
 			(thermal_bridge_width 0.5)
@@
 		(min_thickness 0.25)
 		(filled_areas_thickness no)
-		(fill
+		(fill yes
 			(thermal_gap 0.5)
 			(thermal_bridge_width 0.5)

Commit message: 022825 sync
Parts:
- removed J1: Screw_Terminal_01x04, TerminalBlock:TerminalBlock_bornier-4_P5.08mm
- added J2: 1899003, 4-pos-terminal:PHOENIX_1899003, F.Cu at (210.4, 126.0)
- moved BT1 5.49 mm to (194.3, 70.2)
