File: DAQ_design/v0.2.1/CAD/v0.2.1/_autosave-v0.2.1.kicad_sch (KiCad schematic)
At the start: 37 parts, among them J2 1899003, U1 Teensy4.0, U2 L293D, U3 PC817, U5 PC817, U6 PC817, U7 74HC165

Commit message: 022825 sync
Parts:
- J2: footprint 1899003:PHOENIX_1899003 -> 4-pos-terminal:PHOENIX_1899003
Changed lines of the file:
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@@
 			)
 		)
-		(property "Footprint" "1899003:PHOENIX_1899003"
+		(property "Footprint" "4-pos-terminal:PHOENIX_1899003"
 			(at 154.94 175.26 0)
 			(effects
