File: DAQ_design/Assisi/v0.1/CAD/biphasic_v0.2.1/biphasic_resized/biphasic_resized.kicad_pcb (KiCad board)
At the start: 2 copper layers, 119 x 75 mm, 25 parts, among them Q1 BC549, Q2 IRF9540N, Q3 IRF540N, Q4 BC549, Q5 IRF540N, Q6 IRF9540N

Commit message: pcb
Parts:
- removed ADC: ADS1115IDGS, ads1115module_silkscreen:Adafruit_ADS1115
- removed D1, D2, D3, D4: D_Zener, Diode_THT:D_DO-35_SOD27_P7.62mm_Horizontal
- removed Terminal Out: Screw_Terminal_01x07, TerminalBlock_Phoenix:TerminalBlock_Phoenix_MKDS-1,5-7-5.08_1x07_P5.08mm_Horizontal
Routing:
- net AIN0: track 49.3 -> 0.07 mm
