File: DAQ_design/Assisi/v0.1/CAD/biphasic_v0.2.1/biphasic_resized/biphasic_resized.kicad_sch (KiCad schematic)
At the start: 26 parts, among them Q1 BC549, Q2 IRF9540N, Q3 IRF540N, Q4 BC549, Q5 IRF540N, Q6 IRF9540N

Commit message: pcb
Changed lines of the file:
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@@
 (kicad_sch
-	(version 20231120)
+	(version 20250114)
 	(generator "eeschema")
-	(generator_version "8.0")
+	(generator_version "9.0")
 	(paper "A4")
 	(junction
@@
 		)
 	)
+	(embedded_fonts no)
 )
