File: DAQ_design/Assisi/v0.2.2/EDA/assisi_v0.2.2.kicad_pcb (KiCad board)
At the start: 2 copper layers, 72.5 x 74 mm, 19 parts, among them Q1 BC549, Q2 IRF9540N, Q3 IRF540N, Q4 BC549, Q5 IRF540N, Q6 IRF9540N

Commit message: upload iteration 1
Parts:
- moved H2 80.2 mm to (97.0, 70.3)
- moved H3 78.2 mm to (96.5, 56.3)
- moved G2 70.8 mm to (263.5, 96.5)
- moved G7 70.6 mm to (228.0, 43.0)
- moved Microcontroller 47.9 mm to (199.5, 72.3), turned to 0 degrees
- moved VPP 30.0 mm to (208.5, 52.5), turned to -90 degrees
- moved BiPhasic_out1 22.9 mm to (161.4, 75.4)
- moved R3 19.7 mm to (198.5, 59.7)
- moved Q1 19.7 mm to (189.5, 57.2)
- moved Q2 19.7 mm to (177.5, 60.2)
- moved Q3 19.7 mm to (164.5, 58.2)
- moved R2 19.7 mm to (178.5, 56.2)
- moved Q4 19.5 mm to (189.5, 43.5)
- moved Q5 19.5 mm to (164.5, 43.5)
- moved Q6 19.5 mm to (177.5, 41.5)
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Routing:
- net SN: track 24.5 -> 14.6 mm
- net SP: track 25.1 -> 16.3 mm
- net LOGIC1: track 43.5 -> 47.7 mm
Other:
- board size 72.5 x 74 mm -> 74 x 80 mm
- board text added: "Assisi V0.2.2 07/07/2026"
- board text removed: "Assisi V0.2.2 07/03/2026"
